File: STM32WB breakout board/STM32WB breakout board.kicad_pcb (KiCad board)
At the start: 2 copper layers, 4 parts, among them J1 TSW-133-07-H-S, J2 TSW-133-07-H-S, U1 STM32WB15CCU6

Commit message: Temp
Parts:
- added C2: 10 pF, Capacitor_THT:C_Radial_D5.0mm_H11.0mm_P2.00mm, F.Cu at (218.0, 99.0)
- added C3: 10 pF, Capacitor_THT:C_Radial_D5.0mm_H11.0mm_P2.00mm, F.Cu at (218.0, 105.6)
- added Y1: 32.768 kHz, Crystal:Crystal_HC49-U_Vertical, F.Cu at (223.5, 96.5)
- added Y2: 32 MHz, Crystal:Crystal_SMD_2016-4Pin_2.0x1.6mm, F.Cu at (154.2, 103.6)
Connections:
- J1 pad 33: /OSC_IN -> unconnected-(J1-Pad33)
- J2 pad 01: /OSC_OUT -> unconnected-(J2-Pad01)
- J2 pad 22: /OSC32_OUT -> unconnected-(J2-Pad22)
- J2 pad 23: /OSC32_IN -> unconnected-(J2-Pad23)
Routing:
- net /OSC32_IN: track 42.2 -> 0.00 mm
- net /OSC32_OUT: track 40.9 -> 0.00 mm
Other:
- board text removed: "OSC32_OUT"

Commit message: Temp
Parts:
- Y1: footprint Crystal:Crystal_HC49-U_Vertical -> Crystal:Crystal_C38-LF_D3.0mm_L8.0mm_Vertical
- moved Y2 2.54 mm to (154.2, 101.0), turned to 180 degrees
- moved U1 0.12 mm to (148.1, 94.9)
Routing:
- net /OSC_OUT: track 54.2 -> 0.00 mm
- net GND: track 93.7 -> 42.7 mm
- net /OSC_IN: track 49.1 -> 0.00 mm
- net (no net): track 0.00 -> 12.7 mm
- net /VDDRF: track 52.5 -> 51.8 mm
Other:
- board text removed: "OSC_IN"
- board text removed: "OSC_OUT"

Commit message: Temp
Parts:
- added C4: 100nF, Capacitor_THT:C_Radial_D5.0mm_H11.0mm_P2.00mm, F.Cu at (168.2, 38.1)
- added D1: BAT54W, Package_TO_SOT_SMD:SOT-323_SC-70, F.Cu at (146.3, 48.3)
- added JP1: SolderJumper_2_Open, Resistor_SMD:R_1812_4532Metric, F.Cu at (129.5, 35.6)
- added R2: 10k, Resistor_SMD:R_1218_3246Metric_Pad1.22x4.75mm_HandSolder, F.Cu at (146.7, 26.6)
- added R3: 100k, Resistor_SMD:R_1218_3246Metric_Pad1.22x4.75mm_HandSolder, F.Cu at (158.5, 25.4)
Connections:
- net /PA13 renamed /SWDIO
- net /PA14 renamed /SWCLK
- J1 pad 31: /AT1 -> unconnected-(J1-Pad31)
- J1 pad 32: /AT0 -> unconnected-(J1-Pad32)
- J2 pad 18: /NRST -> /NRST_Pin
- J2 pad 21: /BOOT0 -> unconnected-(J2-Pad21)
- U1 pad 26: /AT0 -> unconnected-(U1-AT0-Pad26)
- U1 pad 27: /AT1 -> unconnected-(U1-AT1-Pad27)
Routing:
- net (no net): track 12.7 -> 107.5 mm
- net /AT0: track 47.8 -> 0.00 mm
- net /AT1: track 47.0 -> 0.00 mm

Commit message: Temp
Parts:
- added C5: 100nF, Capacitor_THT:C_Radial_D5.0mm_H11.0mm_P2.00mm, F.Cu at (63.6, 89.6)
- added C6: 100 pF, Capacitor_THT:C_Radial_D5.0mm_H11.0mm_P2.00mm, F.Cu at (63.6, 96.2)
- added U2: STM32WB15CCU6, STM32WB15CCU6:QFPN_15CCU6_STM, F.Cu at (72.7, 91.2)
Connections:
- J2 pad 02: /VDDRF -> unconnected-(J2-Pad02)
- J2 pad 03: GND -> unconnected-(J2-Pad03)
Routing:
- net unconnected-(J2-Pad02): track 0.00 -> 51.8 mm
- net /VDDRF: track 51.8 -> 0.00 mm

Commit message: Temp
Parts:
- removed U2: STM32WB15CCU6, STM32WB15CCU6:QFPN_15CCU6_STM
- added C7: GRM1555C1HR30WA01D, GRM1555C1HR30WA01D:CAPC1005X55N, F.Cu at (78.3, 41.0)
- added C9: GRM1555C1HR80BA01D, GRM1555C1HR80BA01D:CAPC1005X55N, F.Cu at (78.3, 43.2)
- added FL1: DLF162500LT-5028A1, KiCad:DLF162500LT5028A1, F.Cu at (80.7, 71.1)
- added L1: LQG15HS2N7S02D, LQG15HS2N7S02D:INDC1005X55N, F.Cu at (84.3, 53.3)
- moved C6 2.87 mm to (63.6, 99.1)
Connections:
- C5 pad 1: +3V3 -> 3V3
- C6 pad 1: +3V3 -> 3V3
- JP1 pad 1: +3.3V -> 3V3
- R3 pad 1: +3.3V -> 3V3
- U1 pad 22: GND -> /VSSRF
Routing:
- net unconnected-(J2-Pad02): track 51.8 -> 0.00 mm
Other:
- board text removed: "VDDRF"

Commit message: Temp
Connections:
- FL1 pad 3: unconnected-(FL1-OUT-Pad3) -> Net-(FL1-OUT)
Changed lines of the file:
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@@
   (net 79 "/ RF Section/RF1")
   (net 80 "Net-(FL1-IN)")
-  (net 81 "unconnected-(FL1-OUT-Pad3)")
+  (net 81 "Net-(FL1-OUT)")
   (footprint "Package_TO_SOT_SMD:SOT-323_SC-70" (layer "F.Cu")
     (at 146.32 48.26)
@@
         (effects (font (size 1 1) (thickness 0.15)))
     )
+    (fp_text user "*" (at -4.491 -3.000756) (layer "F.SilkS")
+        (effects (font (size 1 1) (thickness 0.15)))
+    )
     (fp_text user "*" (at -4.491 -3.000756 unlocked) (layer "F.SilkS")
         (effects (font (size 1 1) (thickness 0.15)))
     )
-    (fp_text user "*" (at -4.491 -3.000756) (layer "F.SilkS")
+    (fp_text user "*" (at -3.048 -3.000756) (layer "F.Fab")
         (effects (font (size 1 1) (thickness 0.15)))
     )
     (fp_text user "*" (at -3.048 -3.000756 unlocked) (layer "F.Fab")
-        (effects (font (size 1 1) (thickness 0.15)))
-    )
-    (fp_text user "*" (at -3.048 -3.000756) (layer "F.Fab")
         (effects (font (size 1 1) (thickness 0.15)))
     )
@@
       (net 43 "GND") (pinfunction "GND_1") (pintype "passive"))
     (pad "3" smd rect (at 0.613 0) (size 0.275 0.7) (layers "F.Cu" "F.Paste" "F.Mask")
-      (net 81 "unconnected-(FL1-OUT-Pad3)") (pinfunction "OUT") (pintype "passive"))
+      (net 81 "Net-(FL1-OUT)") (pinfunction "OUT") (pintype "passive"))
     (pad "4" smd rect (at 0 -0.227 90) (size 0.245 0.45) (layers "F.Cu" "F.Paste" "F.Mask")
       (net 43 "GND") (pinfunction "GND_2") (pintype "passive"))

Commit message: Temp
Parts:
- added J3: RSP-122811-02, RSP-122811-02:SAMTEC_RSP-122811-02, F.Cu at (123.5, 55.9)
Changed lines of the file:
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@@
+        (effects (font (size 1 1) (thickness 0.15)))
+    )
+    (fp_text user "${REFERENCE}" (at 0 0 unlocked) (layer "F.Fab")
         (effects (font (size 1 1) (thickness 0.15)))
     )
     (fp_text user "*" (at -3.048 -3.000756 unlocked) (layer "F.Fab")
-        (effects (font (size 1 1) (thickness 0.15)))
-    )
-    (fp_text user "${REFERENCE}" (at 0 0 unlocked) (layer "F.Fab")
         (effects (font (size 1 1) (thickness 0.15)))
     )
@@
       (net 42 "/EPAD") (pinfunction "EPAD") (pintype "power_out"))
   )
+  (footprint "RSP-122811-02:SAMTEC_RSP-122811-02" (layer "F.Cu")
+    (at 123.46 55.88)
+    (property "Availability" "In Stock")
+    (property "Check_prices" "https://www.snapeda.com/parts/RSP-122811-02/Samtec+Inc./view-part/?ref=eda")
+    (property "Description" "\nIPEX MHFIII Connector Receptacle, Male Pin 50 Ohms Surface Mount Solder\n")
+    (property "MANUFACTURER" "SAMTEC")
+    (property "MF" "Samtec Inc.")
+    (property "MP" "RSP-122811-02")
+    (property "PARTREV" "")
+    (property "Package" "None")
+    (property "Price" "None")
+    (property "Purchase-URL" "https://www.snapeda.com/api/url_track_click_mouser/?unipart_id=2771725&manufacturer=Samtec Inc.&part_name=RSP-122811-02&search_term=ipex connector")
+    (property "STANDARD" "Manufacturer recommendations")
+    (property "Sheetfile" " RF Section_sch.kicad_sch")
+    (property "Sheetname" " RF Section")
+    (property "SnapEDA_Link" "https://www.snapeda.com/parts/RSP-122811-02/Samtec+Inc./view-part/?ref=snap")
+    (attr smd)
+    (fp_text reference "J3" (at 0.475085 -2.635435) (layer "F.SilkS")
+        (effects (font (size 1.000165 1.000165) (thickness 0.15)))
+    )
+    (fp_text value "RSP-122811-02" (at 10.10127 2.36531) (layer "F.Fab")
+        (effects (font (size 1.000126 1.000126) (thickness 0.15)))
+    )
+    (fp_line (start -0.93 0.93) (end -0.93 1)
+      (stroke (width 0.127) (type solid)) (layer "F.SilkS"))
+    (fp_line (start -0.93 1) (end -0.43 1)
+      (stroke (width 0.127) (type solid)) (layer "F.SilkS"))
+    (fp_line (start -0.92 -0.9) (end -0.43 -0.9)
+      (stroke (width 0.127) (type solid)) (layer "F.SilkS"))
+    (fp_line (start 0.43 -0.9) (end 0.92 -0.9)
+      (stroke (width 0.127) (type solid)) (layer "F.SilkS"))
+    (fp_line (start 0.43 1) (end 0.93 1)
+      (stroke (width 0.127) (type solid)) (layer "F.SilkS"))
+    (fp_line (start 0.93 1) (end 0.93 0.93)
+      (stroke (width 0.127) (type solid)) (layer "F.SilkS"))
+    (fp_line (start -1.55 -1.55) (end 1.55 -1.55)
+      (stroke (width 0.05) (type solid)) (layer "F.CrtYd"))
+    (fp_line (start -1.55 1.55) (end -1.55 -1.55)
+      (stroke (width 0.05) (type solid)) (layer "F.CrtYd"))
+    (fp_line (start 1.55 -1.55) (end 1.55 1.55)
+      (stroke (width 0.05) (type solid)) (layer "F.CrtYd"))
+    (fp_line (start 1.55 1.55) (end -1.55 1.55)
+      (stroke (width 0.05) (type solid)) (layer "F.CrtYd"))
+    (fp_line (start -0.925 -0.9) (end 0.925 -0.9)
+      (stroke (width 0.127) (type solid)) (layer "F.Fab"))
+    (fp_line (start -0.925 1) (end -0.925 -0.9)
+      (stroke (width 0.127) (type solid)) (layer "F.Fab"))
+    (fp_line (start 0.925 -0.9) (end 0.925 1)
+      (stroke (width 0.127) (type solid)) (layer "F.Fab"))
+    (fp_line (start 0.925 1) (end -0.925 1)
+      (stroke (width 0.127) (type solid)) (layer "F.Fab"))
+    (pad "1" smd rect (at 0 0.975 90) (size 0.65 0.5) (layers "F.Cu" "F.Paste" "F.Mask")
+      (net 81 "Net-(FL1-OUT)") (pinfunction "SIGNAL") (pintype "power_in") (solder_mask_margin 0.102))
+    (pad "2" smd rect (at -1 0 90) (size 1.5 0.6) (layers "F.Cu" "F.Paste" "F.Mask")
+      (net 43 "GND") (pinfunction "GND") (pintype "power_in") (solder_mask_margin 0.102))
+    (pad "3" smd rect (at 0 -1.025 90) (size 0.55 0.5) (layers "F.Cu" "F.Paste" "F.Mask")
+      (net 43 "GND") (pinfunction "GND") (pintype "power_in") (solder_mask_margin 0.102))
+    (pad "4" smd rect (at 1 0 90) (size 1.5 0.6) (layers "F.Cu" "F.Paste" "F.Mask")
+      (net 43 "GND") (pinfunction "GND") (pintype "power_in") (solder_mask_margin 0.102))
+  )
   (footprint "TSW-133-07-H-S:SAMTEC_TSW-133-07-H-S" (layer "F.Cu")

Commit message: Temp
Parts:
- added C8: 100nF, Capacitor_THT:C_Radial_D5.0mm_H11.0mm_P2.00mm, F.Cu at (147.9, 134.6)
- C1: value C_Polarized -> 4.7 uF; footprint Capacitor_THT:CP_Radial_D5.0mm_P2.50mm -> Capacitor_THT:C_Radial_D5.0mm_H11.0mm_P2.00mm
- moved C1 9.58 mm to (219.0, 81.3)
Connections:
- net / RF Section/RF1 renamed / RF & Power /RF1
- C1 pad 1: unconnected-(C1-Pad1) -> 3V3
- C1 pad 2: unconnected-(C1-Pad2) -> GND
