File: STM32WB breakout board/STM32WB breakout board.kicad_pcb (KiCad board)
At the start: 2 copper layers, 70 x 80 mm, 42 parts, among them J1 Conn_02x10_Counter_Clockwise, J2 Conn_02x10_Counter_Clockwise, J3 RSP-122811-02, J4 Conn_02x10_Counter_Clockwise, J5 Conn_02x10_Counter_Clockwise, J6 USB_B_Micro, U1 STM32WB15CCU6, U2 LD1117S33TR_SOT223, X1 32 MHz, X2 32.768 kHz

Commit message: pcb updated
Parts:
- moved C11 100.4 mm to (155.7, 91.4), turned to 90 degrees
- moved C7 100.0 mm to (164.6, 91.7), turned to 90 degrees
- moved C9 87.0 mm to (158.9, 91.4), turned to 90 degrees
- moved C10 78.0 mm to (157.4, 91.4), turned to 90 degrees
- moved C19 46.5 mm to (149.6, 119.0), turned to -90 degrees
- moved C20 39.8 mm to (160.1, 111.2)
- moved U2 39.7 mm to (152.8, 111.2)
- moved C8 32.0 mm to (160.4, 91.4), turned to 90 degrees
- moved X1 7.95 mm to (159.2, 129.7)
- moved X2 7.51 mm to (159.2, 120.3)
- moved J3 5.24 mm to (128.6, 56.7)
- moved J2 4.57 mm to (126.3, 74.2)
- moved J4 4.57 mm to (126.1, 105.6)
- moved S2 4.20 mm to (123.7, 63.1)
- moved U1 2.36 mm to (150.1, 93.7)
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Other:
- board size 70 x 80 mm -> 62 x 80 mm

Commit message: MCU Symbol updated
Parts:
- U1: footprint STM32WB15CCU6:QFPN_15CCU6_STM -> Package_DFN_QFN:QFN-48-1EP_7x7mm_P0.5mm_EP5.6x5.6mm
Connections:
- net /PB8/SCL renamed /SCL/PB8
- net /PB9/SDA renamed /SDA/PB9
- U1 pad 40: /VDDUSB -> 3V3

Commit message: PCB updated
Parts:
- moved C12 111.4 mm to (143.4, 99.6), turned to 90 degrees
- moved C20 22.0 mm to (141.0, 121.9), turned to 90 degrees
- moved C7 12.4 mm to (160.3, 103.3)
- moved C8 12.3 mm to (156.2, 103.0)
- moved C9 12.3 mm to (154.7, 103.0)
- moved C10 12.3 mm to (153.2, 103.0)
- moved R1 12.2 mm to (186.6, 43.6)
- moved C14 12.2 mm to (151.1, 70.6)
- moved C19 12.2 mm to (145.7, 130.5)
- moved D2 12.2 mm to (136.9, 125.0)
- moved J1 12.2 mm to (174.2, 84.8)
- moved J3 12.2 mm to (124.7, 68.3)
- moved J5 12.2 mm to (174.4, 114.5)
- moved S1 12.2 mm to (166.6, 72.1)
- moved S2 12.2 mm to (119.7, 74.7)
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
Commit message: PCB updated
Parts:
- moved J1 51.9 mm to (122.3, 85.8)
- moved J2 51.9 mm to (174.2, 84.8)
- moved D1 44.9 mm to (138.2, 104.5), turned to 90 degrees
- moved C18 44.1 mm to (141.1, 105.0), turned to 90 degrees
Changed lines of the file:
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@@
   )
   (footprint "Package_TO_SOT_SMD:SOT-323_SC-70" (layer "F.Cu")
-    (at 142.374 59.818)
+    (at 138.225 104.5 90)
     (descr "SOT-323, SC-70")
     (tags "SOT-323 SC-70")
@@
     (property "ki_keywords" "schottky diode")
     (attr smd)
-    (fp_text reference "D1" (at -0.05 -1.95) (layer "F.SilkS")
+    (fp_text reference "D1" (at 2.65 0 90) (layer "F.SilkS")
         (effects (font (size 1 1) (thickness 0.15)))
     )
-    (fp_text value "BAT54W" (at -0.05 2.05) (layer "F.Fab")
+    (fp_text value "BAT54W" (at -0.05 2.05 90) (layer "F.Fab")
         (effects (font (size 1 1) (thickness 0.15)))
     )
-    (fp_text user "${REFERENCE}" (at 0 0 90) (layer "F.Fab")
+    (fp_text user "${REFERENCE}" (at 0 0) (layer "F.Fab")
         (effects (font (size 0.5 0.5) (thickness 0.075)))
     )
@@
     (fp_line (start 0.67 1.1) (end -0.68 1.1)
       (stroke (width 0.1) (type solid)) (layer "F.Fab"))
-    (pad "1" smd rect (at -1 -0.65 270) (size 0.45 0.7) (layers "F.Cu" "F.Paste" "F.Mask")
+    (pad "1" smd rect (at -1 -0.65) (size 0.45 0.7) (layers "F.Cu" "F.Paste" "F.Mask")
       (net 4 "/NRST") (pinfunction "A") (pintype "passive"))
-    (pad "2" smd rect (at -1 0.65 270) (size 0.45 0.7) (layers "F.Cu" "F.Paste" "F.Mask")
+    (pad "2" smd rect (at -1 0.65) (size 0.45 0.7) (layers "F.Cu" "F.Paste" "F.Mask")
       (net 16 "unconnected-(D1-NC-Pad2)") (pinfunction "NC") (pintype "no_connect"))
-    (pad "3" smd rect (at 1 0 270) (size 0.45 0.7) (layers "F.Cu" "F.Paste" "F.Mask")
+    (pad "3" smd rect (at 1 0) (size 0.45 0.7) (layers "F.Cu" "F.Paste" "F.Mask")
       (net 17 "/NRST_Pin") (pinfunction "K") (pintype "passive"))
     (model "${KICAD6_3DMODEL_DIR}/Package_TO_SOT_SMD.3dshapes/SOT-323_SC-70.wrl"
@@
   )
   (footprint "Connector_PinSocket_2.54mm:PinSocket_2x10_P2.54mm_Vertical" (layer "F.Cu")
-    (at 122.334 85.758)
+    (at 174.194 84.808)
     (descr "Through hole straight socket strip, 2x10, 2.54mm pitch, double cols (from Kicad 4.0.7), script generated")
     (tags "Through hole socket strip THT 2x10 2.54mm double row")
@@
   )
   (footprint "Connector_PinSocket_2.54mm:PinSocket_2x10_P2.54mm_Vertical" (layer "F.Cu")
-    (at 174.194 84.808)
+    (at 122.334 85.758)
     (descr "Through hole straight socket strip, 2x10, 2.54mm pitch, double cols (from Kicad 4.0.7), script generated")
     (tags "Through hole socket strip THT 2x10 2.54mm double row")
@@
   )
   (footprint "Capacitor_SMD:C_0402_1005Metric" (layer "F.Cu")
-    (at 164.234 67.438)
+    (at 141.05 105.005 90)
     (descr "Capacitor SMD 0402 (1005 Metric), square (rectangular) end terminal, IPC_7351 nominal, (Body size source: IPC-SM-782 page 76, https://www.pcb-3d.com/wordpress/wp-content/uploads/ipc-sm-782a_amendment_1_and_2.pdf), generated with kicad-footprint-generator")
     (tags "capacitor")
@@
     (property "ki_keywords" "cap capacitor")
     (attr smd)
-    (fp_text reference "C18" (at 0 -1.16) (layer "F.SilkS")
+    (fp_text reference "C18" (at 2.405 0 90) (layer "F.SilkS")
         (effects (font (size 1 1) (thickness 0.15)))
     )
-    (fp_text value "100nF" (at 0 1.16) (layer "F.Fab")
+    (fp_text value "100nF" (at 0 1.16 90) (layer "F.Fab")
         (effects (font (size 1 1) (thickness 0.15)))
     )
-    (fp_text user "${REFERENCE}" (at 0 0) (layer "F.Fab")
+    (fp_text user "${REFERENCE}" (at 0 0 90) (layer "F.Fab")
         (effects (font (size 0.25 0.25) (thickness 0.04)))
     )
@@
     (fp_line (start 0.5 0.25) (end -0.5 0.25)
       (stroke (width 0.1) (type solid)) (layer "F.Fab"))
-    (pad "1" smd roundrect (at -0.48 0) (size 0.56 0.62) (layers "F.Cu" "F.Paste" "F.Mask") (roundrect_rratio 0.25)
+    (pad "1" smd roundrect (at -0.48 0 90) (size 0.56 0.62) (layers "F.Cu" "F.Paste" "F.Mask") (roundrect_rratio 0.25)
       (net 4 "/NRST") (pintype "passive"))
-    (pad "2" smd roundrect (at 0.48 0) (size 0.56 0.62) (layers "F.Cu" "F.Paste" "F.Mask") (roundrect_rratio 0.25)
+    (pad "2" smd roundrect (at 0.48 0 90) (size 0.56 0.62) (layers "F.Cu" "F.Paste" "F.Mask") (roundrect_rratio 0.25)
       (net 30 "GND") (pintype "passive"))
     (model "${KICAD6_3DMODEL_DIR}/Capacitor_SMD.3dshapes/C_0402_1005Metric.wrl"

Commit message: schematic updated
Parts:
- moved L1 84.9 mm to (152.7, 109.1), turned to -90 degrees
- moved L2 73.4 mm to (152.7, 105.7), turned to -90 degrees
- moved C1 52.2 mm to (165.4, 109.0), turned to 90 degrees
- moved C7 1.04 mm to (160.8, 102.5)
- moved C11 0.78 mm to (152.3, 102.5)
- moved C8 0.78 mm to (156.8, 102.5)
- moved C10 0.78 mm to (153.8, 102.5)
- moved C9 0.78 mm to (155.3, 102.5)
Connections:
- C1 pad 1: /RF & Power/VFBSMPS -> /VFBSMPS
- C2 pad 2: /RF & Power/RF1 -> /RF1
- L1 pad 2: /RF & Power/VFBSMPS -> /VFBSMPS
- L2 pad 1: /RF & Power/VLXSMPS -> /VLXSMPS
- L3 pad 1: /RF & Power/RF1 -> /RF1
- U1 pad 23: /VDDRF -> 3V3
- U1 pad 34: /VDDSMPS -> 3V3

Commit message: schematic updated
Parts:
- moved C1 6.19 mm to (159.3, 110.0)
Changed lines of the file:
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@@
   )
   (footprint "LQG15WZ10NJ02D:INDC1006X60N" (layer "F.Cu")
-    (at 152.72 105.7325 -90)
+    (at 152.74 105.722 -90)
     (property "Availability" "In Stock")
     (property "Check_prices" "https://www.snapeda.com/parts/LQG15WZ10NJ02D/Murata+Electronics+North+America/view-part/?ref=eda")
@@
     (property "SnapEDA_Link" "https://www.snapeda.com/parts/LQG15WZ10NJ02D/Murata+Electronics+North+America/view-part/?ref=snap")
     (attr smd)
-    (fp_text reference "L2" (at 0.0025 -0.91 90) (layer "F.SilkS")
+    (fp_text reference "L2" (at -0.002 -1 90) (layer "F.SilkS")
         (effects (font (size 0.393701 0.393701) (thickness 0.15)))
     )
@@
   )
   (footprint "Capacitor_THT:CP_Radial_D5.0mm_P2.00mm" (layer "F.Cu")
-    (at 165.43 109.005113 90)
+    (at 159.32 109.98 90)
     (descr "CP, Radial series, Radial, pin pitch=2.00mm, , diameter=5mm, Electrolytic Capacitor")
     (tags "CP Radial series Radial pin pitch 2.00mm  diameter 5mm Electrolytic Capacitor")
@@
     (property "SnapEDA_Link" "https://www.snapeda.com/parts/LQM21FN100M70L/Murata+Electronics+North+America/view-part/?ref=snap")
     (attr smd)
-    (fp_text reference "L1" (at -0.46 -1.32 90) (layer "F.SilkS")
+    (fp_text reference "L1" (at 0 -1.35 90) (layer "F.SilkS")
         (effects (font (size 0.393701 0.393701) (thickness 0.15)))
     )

Commit message: PCB updated
Parts:
- moved C15 97.3 mm to (139.8, 106.4), turned to 90 degrees
- moved C6 81.6 mm to (141.0, 103.8), turned to 180 degrees
- moved C5 81.3 mm to (141.0, 102.6), turned to 180 degrees
- moved C16 70.3 mm to (141.2, 106.3), turned to 90 degrees
- moved C18 6.57 mm to (134.9, 102.8)
- moved D1 6.05 mm to (132.5, 102.5)
Changed lines of the file:
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@@
   )
   (footprint "Package_TO_SOT_SMD:SOT-323_SC-70" (layer "F.Cu")
-    (at 138.225 104.5 90)
+    (at 132.5 102.54 90)
     (descr "SOT-323, SC-70")
     (tags "SOT-323 SC-70")
@@
   )
   (footprint "Capacitor_SMD:C_0402_1005Metric" (layer "F.Cu")
-    (at 88.034 152.328)
+    (at 141.2 106.29 90)
     (descr "Capacitor SMD 0402 (1005 Metric), square (rectangular) end terminal, IPC_7351 nominal, (Body size source: IPC-SM-782 page 76, https://www.pcb-3d.com/wordpress/wp-content/uploads/ipc-sm-782a_amendment_1_and_2.pdf), generated with kicad-footprint-generator")
     (tags "capacitor")
@@
     (property "ki_keywords" "cap capacitor")
     (attr smd)
-    (fp_text reference "C16" (at 0 -1.16) (layer "F.SilkS")
+    (fp_text reference "C16" (at -2.4 0 90) (layer "F.SilkS")
         (effects (font (size 1 1) (thickness 0.15)))
     )
-    (fp_text value "10 nF" (at 0 1.16) (layer "F.Fab")
+    (fp_text value "10 nF" (at 0 1.16 90) (layer "F.Fab")
         (effects (font (size 1 1) (thickness 0.15)))
     )
-    (fp_text user "${REFERENCE}" (at 0 0) (layer "F.Fab")
+    (fp_text user "${REFERENCE}" (at 0 0 90) (layer "F.Fab")
         (effects (font (size 0.25 0.25) (thickness 0.04)))
     )
@@
     (fp_line (start 0.5 0.25) (end -0.5 0.25)
       (stroke (width 0.1) (type solid)) (layer "F.Fab"))
-    (pad "1" smd roundrect (at -0.48 0) (size 0.56 0.62) (layers "F.Cu" "F.Paste" "F.Mask") (roundrect_rratio 0.25)
+    (pad "1" smd roundrect (at -0.48 0 90) (size 0.56 0.62) (layers "F.Cu" "F.Paste" "F.Mask") (roundrect_rratio 0.25)
       (net 29 "3V3") (pintype "passive"))
-    (pad "2" smd roundrect (at 0.48 0) (size 0.56 0.62) (layers "F.Cu" "F.Paste" "F.Mask") (roundrect_rratio 0.25)
+    (pad "2" smd roundrect (at 0.48 0 90) (size 0.56 0.62) (layers "F.Cu" "F.Paste" "F.Mask") (roundrect_rratio 0.25)
       (net 28 "GND") (pintype "passive"))
     (model "${KICAD6_3DMODEL_DIR}/Capacitor_SMD.3dshapes/C_0402_1005Metric.wrl"
@@
   )
   (footprint "Capacitor_SMD:C_0402_1005Metric_Pad0.74x0.62mm_HandSolder" (layer "F.Cu")
-    (at 232.754 77.598)
+    (at 139.78 106.3625 90)
     (descr "Capacitor SMD 0402 (1005 Metric), square (rectangular) end terminal, IPC_7351 nominal with elongated pad for handsoldering. (Body size source: IPC-SM-782 page 76, https://www.pcb-3d.com/wordpress/wp-content/uploads/ipc-sm-782a_amendment_1_and_2.pdf), generated with kicad-footprint-generator")
     (tags "capacitor handsolder")
@@
     (property "ki_keywords" "cap capacitor")
     (attr smd)
-    (fp_text reference "C15" (at 0 -1.16) (layer "F.SilkS")
+    (fp_text reference "C15" (at -2.6025 0 90) (layer "F.SilkS")
         (effects (font (size 1 1) (thickness 0.15)))
     )
-    (fp_text value "1 uF" (at 0 1.16) (layer "F.Fab")
+    (fp_text value "1 uF" (at 0 1.16 90) (layer "F.Fab")
         (effects (font (size 1 1) (thickness 0.15)))
     )
-    (fp_text user "${REFERENCE}" (at 0 0) (layer "F.Fab")
+    (fp_text user "${REFERENCE}" (at 0 0 90) (layer "F.Fab")
         (effects (font (size 0.25 0.25) (thickness 0.04)))
     )
@@
     (fp_line (start 0.5 0.25) (end -0.5 0.25)
       (stroke (width 0.1) (type solid)) (layer "F.Fab"))
-    (pad "1" smd roundrect (at -0.5675 0) (size 0.735 0.62) (layers "F.Cu" "F.Paste" "F.Mask") (roundrect_rratio 0.25)
+    (pad "1" smd roundrect (at -0.5675 0 90) (size 0.735 0.62) (layers "F.Cu" "F.Paste" "F.Mask") (roundrect_rratio 0.25)
       (net 29 "3V3") (pintype "passive"))
-    (pad "2" smd roundrect (at 0.5675 0) (size 0.735 0.62) (layers "F.Cu" "F.Paste" "F.Mask") (roundrect_rratio 0.25)
+    (pad "2" smd roundrect (at 0.5675 0 90) (size 0.735 0.62) (layers "F.Cu" "F.Paste" "F.Mask") (roundrect_rratio 0.25)
       (net 28 "GND") (pintype "passive"))
     (model "${KICAD6_3DMODEL_DIR}/Capacitor_SMD.3dshapes/C_0402_1005Metric.wrl"
@@
   )
   (footprint "Capacitor_SMD:C_0402_1005Metric" (layer "F.Cu")
-    (at 59.663001 101.198308)
+    (at 140.98 102.61 180)
     (descr "Capacitor SMD 0402 (1005 Metric), square (rectangular) end terminal, IPC_7351 nominal, (Body size source: IPC-SM-782 page 76, https://www.pcb-3d.com/wordpress/wp-content/uploads/ipc-sm-782a_amendment_1_and_2.pdf), generated with kicad-footprint-generator")
     (tags "capacitor")
@@
     (property "ki_keywords" "cap capacitor")
     (attr smd)
-    (fp_text reference "C5" (at 0 -1.16) (layer "F.SilkS")
+    (fp_text reference "C5" (at 2.07 0.01) (layer "F.SilkS")
         (effects (font (size 1 1) (thickness 0.15)))
     )
@@
     (fp_line (start 0.5 0.25) (end -0.5 0.25)
       (stroke (width 0.1) (type solid)) (layer "F.Fab"))
-    (pad "1" smd roundrect (at -0.48 0) (size 0.56 0.62) (layers "F.Cu" "F.Paste" "F.Mask") (roundrect_rratio 0.25)
+    (pad "1" smd roundrect (at -0.48 0 180) (size 0.56 0.62) (layers "F.Cu" "F.Paste" "F.Mask") (roundrect_rratio 0.25)
       (net 1 "/OSC32_IN") (pintype "passive"))
-    (pad "2" smd roundrect (at 0.48 0) (size 0.56 0.62) (layers "F.Cu" "F.Paste" "F.Mask") (roundrect_rratio 0.25)
+    (pad "2" smd roundrect (at 0.48 0 180) (size 0.56 0.62) (layers "F.Cu" "F.Paste" "F.Mask") (roundrect_rratio 0.25)
       (net 28 "GND") (pintype "passive"))
     (model "${KICAD6_3DMODEL_DIR}/Capacitor_SMD.3dshapes/C_0402_1005Metric.wrl"
@@
   )
   (footprint "Capacitor_SMD:C_0402_1005Metric" (layer "F.Cu")
-    (at 59.663001 110.618)
+    (at 140.97 103.85 180)
     (descr "Capacitor SMD 0402 (1005 Metric), square (rectangular) end terminal, IPC_7351 nominal, (Body size source: IPC-SM-782 page 76, https://www.pcb-3d.com/wordpress/wp-content/uploads/ipc-sm-782a_amendment_1_and_2.pdf), generated with kicad-footprint-generator")
     (tags "capacitor")
@@
     (property "ki_keywords" "cap capacitor")
     (attr smd)
-    (fp_text reference "C6" (at 0 -1.16) (layer "F.SilkS")
+    (fp_text reference "C6" (at 2.04 0.01) (layer "F.SilkS")
         (effects (font (size 1 1) (thickness 0.15)))
     )
@@
     (fp_line (start 0.5 0.25) (end -0.5 0.25)
       (stroke (width 0.1) (type solid)) (layer "F.Fab"))
-    (pad "1" smd roundrect (at -0.48 0) (size 0.56 0.62) (layers "F.Cu" "F.Paste" "F.Mask") (roundrect_rratio 0.25)
+    (pad "1" smd roundrect (at -0.48 0 180) (size 0.56 0.62) (layers "F.Cu" "F.Paste" "F.Mask") (roundrect_rratio 0.25)
       (net 2 "/OSC32_OUT") (pintype "passive"))
-    (pad "2" smd roundrect (at 0.48 0) (size 0.56 0.62) (layers "F.Cu" "F.Paste" "F.Mask") (roundrect_rratio 0.25)
+    (pad "2" smd roundrect (at 0.48 0 180) (size 0.56 0.62) (layers "F.Cu" "F.Paste" "F.Mask") (roundrect_rratio 0.25)
       (net 28 "GND") (pintype "passive"))
     (model "${KICAD6_3DMODEL_DIR}/Capacitor_SMD.3dshapes/C_0402_1005Metric.wrl"
@@
   )
   (footprint "Capacitor_SMD:C_0402_1005Metric" (layer "F.Cu")
-    (at 141.05 105.005 90)
+    (at 134.88 102.76 90)
     (descr "Capacitor SMD 0402 (1005 Metric), square (rectangular) end terminal, IPC_7351 nominal, (Body size source: IPC-SM-782 page 76, https://www.pcb-3d.com/wordpress/wp-content/uploads/ipc-sm-782a_amendment_1_and_2.pdf), generated with kicad-footprint-generator")
     (tags "capacitor")

Commit message: PCB updated
Parts:
- moved C4 47.9 mm to (149.5, 95.2)
Changed lines of the file:
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@@
   )
   (footprint "Capacitor_THT:CP_Radial_D5.0mm_P2.00mm" (layer "F.Cu")
-    (at 164.234 49.658)
+    (at 149.52 95.22)
     (descr "CP, Radial series, Radial, pin pitch=2.00mm, , diameter=5mm, Electrolytic Capacitor")
     (tags "CP Radial series Radial pin pitch 2.00mm  diameter 5mm Electrolytic Capacitor")
