File: STM32WB breakout board/STM32WB breakout board.kicad_sch (KiCad schematic)
At the start: 12 parts, among them J1 TSW-133-07-H-S, J2 TSW-133-07-H-S, U1 STM32WB15CCU6, Y1 32.768 kHz, Y2 32 MHz

Commit message: Temp
Other:
- sheet  RF Section renamed  RF & Power 
- removed sheet Power section
- sheet  RF & Power  ports: added VDDSMPS; removed none
Changed lines of the file:
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@@
+    (stroke (width 0) (type default))
+  )
+  (wire (pts (xy 187.452 71.882) (xy 192.024 71.882))
     (stroke (width 0) (type default))
   )
@@
     (stroke (width 0) (type default))
   )
-  (wire (pts (xy 181.356 72.644) (xy 191.516 72.644))
+  (wire (pts (xy 188.468 74.422) (xy 192.024 74.422))
     (stroke (width 0) (type default))
   )
@@
     (stroke (width 0) (type default))
   )
+  (wire (pts (xy 187.452 72.644) (xy 187.452 71.882))
+    (stroke (width 0) (type default))
+  )
   (wire (pts (xy 181.356 80.264) (xy 191.516 80.264))
     (stroke (width 0) (type default))
@@
     (stroke (width 0) (type default))
   )
+  (wire (pts (xy 181.356 72.644) (xy 187.452 72.644))
+    (stroke (width 0) (type default))
+  )
   (wire (pts (xy 44.45 90.17) (xy 54.864 90.17))
     (stroke (width 0) (type default))
@@
     (stroke (width 0) (type default))
   )
+  (wire (pts (xy 181.356 75.184) (xy 188.468 75.184))
+    (stroke (width 0) (type default))
+  )
   (wire (pts (xy 245.11 55.88) (xy 253.746 55.88))
     (stroke (width 0) (type default))
@@
     (stroke (width 0) (type default))
   )
-  (wire (pts (xy 181.356 75.184) (xy 191.516 75.184))
-    (stroke (width 0) (type default))
-  )
   (wire (pts (xy 105.156 54.864) (xy 115.316 54.864))
     (stroke (width 0) (type default))
@@
   )
   (wire (pts (xy 44.45 97.79) (xy 54.864 97.79))
+    (stroke (width 0) (type default))
+  )
+  (wire (pts (xy 188.468 75.184) (xy 188.468 74.422))
     (stroke (width 0) (type default))
   )
@@
     (effects (font (size 1.27 1.27)) (justify right bottom))
   )
-  (label "VLXSMPS" (at 191.516 75.184 0) (fields_autoplaced)
-    (effects (font (size 1.27 1.27)) (justify left bottom))
-  )
   (label "EPAD" (at 191.516 34.544 0) (fields_autoplaced)
     (effects (font (size 1.27 1.27)) (justify left bottom))
@@
   )
   (label "PA6" (at 105.156 70.104 0) (fields_autoplaced)
-    (effects (font (size 1.27 1.27)) (justify left bottom))
-  )
-  (label "VDDSMPS" (at 191.516 72.644 0) (fields_autoplaced)
     (effects (font (size 1.27 1.27)) (justify left bottom))
   )
@@
     )
   )
+  (hierarchical_label "VLXSMPS" (shape input) (at 192.024 74.422 0) (fields_autoplaced)
+    (effects (font (size 1.27 1.27)) (justify left))
+  )
   (hierarchical_label "VDDRF" (shape input) (at 105.918 90.424 180) (fields_autoplaced)
     (effects (font (size 1.27 1.27)) (justify right))
+  )
+  (hierarchical_label "VDDSMPS" (shape input) (at 192.024 71.882 0) (fields_autoplaced)
+    (effects (font (size 1.27 1.27)) (justify left))
   )
   (hierarchical_label "VSSRF" (shape input) (at 106.172 87.884 180) (fields_autoplaced)
@@
     (stroke (width 0.1524) (type solid))
     (fill (color 0 0 0 0.0000))
-    (property "Sheetname" " RF Section" (at 257.302 125.476 0)
+    (property "Sheetname" " RF & Power " (at 257.302 125.476 0)
       (effects (font (size 1.27 1.27)) (justify left bottom))
     )
@@
       (effects (font (size 1.27 1.27)) (justify left top))
     )
-    (pin "VDDRF" input (at 250.698 129.794 180)
-      (effects (font (size 1.27 1.27)) (justify left))
-    )
-    (pin "VSSRF" input (at 250.698 133.35 180)
-      (effects (font (size 1.27 1.27)) (justify left))
-    )
-    (pin "RF1" input (at 250.698 138.684 180)
+    (pin "VDDRF" input (at 250.698 128.524 180)
+      (effects (font (size 1.27 1.27)) (justify left))
+    )
+    (pin "VSSRF" input (at 250.698 132.334 180)
+      (effects (font (size 1.27 1.27)) (justify left))
+    )
+    (pin "RF1" input (at 250.698 136.398 180)
+      (effects (font (size 1.27 1.27)) (justify left))
+    )
+    (pin "VDDSMPS" input (at 250.698 140.208 180)
       (effects (font (size 1.27 1.27)) (justify left))
     )
@@
       )
     )
-  )
-  (sheet (at 217.424 125.73) (size 25.654 19.05) (fields_autoplaced)
-    (stroke (width 0.1524) (type solid))
-    (fill (color 0 0 0 0.0000))
-    (property "Sheetname" "Power section" (at 217.424 125.0184 0)
-      (effects (font (size 1.27 1.27)) (justify left bottom))
-    )
-    (property "Sheetfile" "Power section_sch.kicad_sch" (at 217.424 145.3646 0)
-      (effects (font (size 1.27 1.27)) (justify left top))
-    )
-    (instances
-      (project "STM32WB breakout board"
-        (path "/29424def-bd0e-47af-8787-429d3d525da1" (page "3"))
-      )
-    )

Commit message: Temp
Parts:
- added C11: 4.7 uF, Capacitor_THT:C_Radial_D5.0mm_H11.0mm_P2.00mm, symbol Device:C
- added C12, C13, C14, C15: 100nF, Capacitor_THT:C_Radial_D5.0mm_H11.0mm_P2.00mm, symbol Device:C
Connections:
- net VBAT is gone; now on net 3V3: J2.24, U1.1 (VBAT)
- net 3V3: now also J1.10, J1.18, J1.23, J2.05, U1.20 (VDD), U1.35 (VDD), U1.48 (VDD), C11.1, C12.1, C13.1, C14.1, C15.1
- net GND: now also C11.2, C12.2, C13.2, C14.2, C15.2; no longer J1.26, U1.32 (VSSSMPS)
- removed net VDD: J1.10, J1.18, J1.23, J2.05, U1.20 (VDD), U1.35 (VDD), U1.40 (VDD), U1.48 (VDD)
- new net VDDUSB: U1.40 (VDD)
- new net VSSSMPS: J1.26, U1.32 (VSSSMPS)
Other:
- sheet  RF & Power  ports: added VFBSMPS, VLXSMPS, VSSSMPS; removed none
- moved on the sheet: J2

Commit message: Temp
Parts:
- added C16: 1 uF, Capacitor_THT:C_Radial_D5.0mm_H11.0mm_P2.00mm, symbol Device:C
- added C17: 10 nF, Capacitor_THT:C_Radial_D5.0mm_H11.0mm_P2.00mm, symbol Device:C
Connections:
- net VDDA is gone; now on net 3V3: J2.17, U1.8 (VDDA)
- net 3V3: now also C16.1, C17.1
- net EPAD: no longer U1.49 (EPAD)
- net GND: now also U1.49 (EPAD), C16.2, C17.2
Other:
- moved on the sheet: C11, C12, C13, C14, C15

Commit message: Temp
Parts:
- removed C13, C14, C15: 100nF, Capacitor_THT:C_Radial_D5.0mm_H11.0mm_P2.00mm, symbol Device:C
- removed C2: 10 pF, Capacitor_THT:C_Radial_D5.0mm_H11.0mm_P2.00mm, symbol Device:C
- added C10, C11, C9: 100nF, Capacitor_SMD:C_0402_1005Metric, symbol Device:C
- added C5: 10 pF, Capacitor_SMD:C_0402_1005Metric, symbol Device:C
- C15: renamed from C16; footprint Capacitor_THT:C_Radial_D5.0mm_H11.0mm_P2.00mm -> Capacitor_SMD:C_0402_1005Metric_Pad0.74x0.62mm_HandSolder
- C16: renamed from C17; footprint Capacitor_THT:C_Radial_D5.0mm_H11.0mm_P2.00mm -> Capacitor_SMD:C_0402_1005Metric
- C6: renamed from C3; footprint Capacitor_THT:C_Radial_D5.0mm_H11.0mm_P2.00mm -> Capacitor_SMD:C_0402_1005Metric
- C8: renamed from C12; footprint Capacitor_THT:C_Radial_D5.0mm_H11.0mm_P2.00mm -> Capacitor_SMD:C_0402_1005Metric
- renumbered C4 to C18, C11 to C7
Connections:
- net 3V3: now also C10.1, C11.1, C9.1; no longer J2.24
- net GND: now also C10.2, C11.2, C5.2, C9.2
- net OSC32_IN: now also C5.1
- net RF1: no longer J2.04
- net VDDSMPS: no longer J1.24
- net VFBSMPS: no longer J1.27
- net VLXSMPS: no longer J1.25
- net VSSSMPS: no longer J1.26
- net EPAD: no longer names the net of J1.09
- net PB0: no longer names the net of U1.28 (PB0)
- net PB0: no longer J1.30
- no-connect marks 2 -> 3
Other:
- moved on the sheet: C15, C16, C18, D1, R3

Commit message: Temp
Parts:
- renumbered Y2 to X1, Y1 to X2
Changed lines of the file:
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@@
   (symbol (lib_id "Device:Crystal") (at 27.432 173.228 180) (unit 1)
     (in_bom yes) (on_board yes) (dnp no)
-    (property "Reference" "Y1" (at 26.162 169.418 0)
+    (property "Reference" "X2" (at 26.162 169.418 0)
       (effects (font (size 1.27 1.27)) (justify right))
     )
@@
       (project "STM32WB breakout board"
         (path "/29424def-bd0e-47af-8787-429d3d525da1"
-          (reference "Y1") (unit 1)
+          (reference "X2") (unit 1)
         )
       )
@@
   (symbol (lib_id "Device:Crystal_GND24") (at 60.198 176.276 90) (unit 1)
     (in_bom yes) (on_board yes) (dnp no)
-    (property "Reference" "Y2" (at 62.992 172.466 90)
+    (property "Reference" "X1" (at 62.992 172.466 90)
       (effects (font (size 1.27 1.27)))
     )
@@
       (project "STM32WB breakout board"
         (path "/29424def-bd0e-47af-8787-429d3d525da1"
-          (reference "Y2") (unit 1)
-        )
-      )
+          (reference "X1") (unit 1)
+        )
+      )

Commit message: Temp
Parts:
- X2: footprint Crystal:Crystal_C38-LF_D3.0mm_L8.0mm_Vertical -> Crystal:Crystal_SMD_2012-2Pin_2.0x1.2mm
Connections:
- net 3V3: no longer J2.17
Changed lines of the file:
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@@
-    (stroke (width 0) (type default))
-  )
-  (wire (pts (xy 43.18 65.786) (xy 53.594 65.786))
     (stroke (width 0) (type default))
   )
@@
   )
   (label "PB9" (at 53.594 60.706 0) (fields_autoplaced)
-    (effects (font (size 1.27 1.27)) (justify left bottom))
-  )
-  (label "VDDA" (at 53.594 65.786 0) (fields_autoplaced)
     (effects (font (size 1.27 1.27)) (justify left bottom))
   )
@@
       (effects (font (size 1.27 1.27)) (justify right))
     )
-    (property "Footprint" "Crystal:Crystal_C38-LF_D3.0mm_L8.0mm_Vertical" (at 27.432 173.228 0)
-      (effects (font (size 1.27 1.27)) hide)
-    )
+    (property "Footprint" "Crystal:Crystal_SMD_2012-2Pin_2.0x1.2mm" (at 27.432 173.228 0)
+      (effects (font (size 1.27 1.27)) hide)
+    )

Commit message: Temp
Parts:
- C18: footprint Capacitor_THT:C_Radial_D5.0mm_H11.0mm_P2.00mm -> Capacitor_SMD:C_0402_1005Metric
Changed lines of the file:
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@@
       (effects (font (size 1.27 1.27)) (justify left))
     )
-    (property "Footprint" "Capacitor_THT:C_Radial_D5.0mm_H11.0mm_P2.00mm" (at 113.2332 181.864 0)
+    (property "Footprint" "Capacitor_SMD:C_0402_1005Metric" (at 113.2332 181.864 0)
       (effects (font (size 1.27 1.27)) hide)
     )

Commit message: Temp
Parts:
- C7: footprint Capacitor_THT:C_Radial_D5.0mm_H11.0mm_P2.00mm -> Capacitor_SMD:C_01005_0402Metric
Changed lines of the file:
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@@
-    )
-  )
-  (symbol (lib_id "Device:C") (at 20.574 137.922 0) (unit 1)
-    (in_bom yes) (on_board yes) (dnp no)
-    (property "Reference" "C7" (at 21.59 135.89 0)
-      (effects (font (size 1.27 1.27)) (justify left))
-    )
-    (property "Value" "4.7 uF" (at 21.336 140.716 0)
-      (effects (font (size 1.27 1.27)) (justify left))
-    )
-    (property "Footprint" "Capacitor_THT:C_Radial_D5.0mm_H11.0mm_P2.00mm" (at 21.5392 141.732 0)
-      (effects (font (size 1.27 1.27)) hide)
-    )
-    (property "Datasheet" "~" (at 20.574 137.922 0)
-      (effects (font (size 1.27 1.27)) hide)
-    )
-    (pin "2")
-    (pin "1")
-    (instances
-      (project "STM32WB breakout board"
-        (path "/29424def-bd0e-47af-8787-429d3d525da1"
-          (reference "C7") (unit 1)
-        )
-        (path "/29424def-bd0e-47af-8787-429d3d525da1/1e4823cc-51de-4557-be75-82cccb133913"
-          (reference "C10") (unit 1)
-        )
-      )
     )
   )
@@
         )
       )
+    )
+  )
+  (symbol (lib_id "Device:C") (at 20.574 137.922 0) (unit 1)
+    (in_bom yes) (on_board yes) (dnp no)
+    (property "Reference" "C7" (at 21.59 135.89 0)
+      (effects (font (size 1.27 1.27)) (justify left))
+    )
+    (property "Value" "4.7 uF" (at 21.336 140.716 0)
+      (effects (font (size 1.27 1.27)) (justify left))
+    )
+    (property "Footprint" "Capacitor_SMD:C_01005_0402Metric" (at 21.5392 141.732 0)
+      (effects (font (size 1.27 1.27)) hide)
+    )
+    (property "Datasheet" "~" (at 20.574 137.922 0)
+      (effects (font (size 1.27 1.27)) hide)
+    )
+    (pin "2")
+    (pin "1")
+    (instances
+      (project "STM32WB breakout board"
+        (path "/29424def-bd0e-47af-8787-429d3d525da1"
+          (reference "C7") (unit 1)
+        )
+        (path "/29424def-bd0e-47af-8787-429d3d525da1/1e4823cc-51de-4557-be75-82cccb133913"
+          (reference "C17") (unit 1)
+        )
+      )
