File: STM32WB breakout board/STM32WB breakout board.kicad_sch (KiCad schematic)
At the start: 19 parts, among them J1 TSW-133-07-H-S, J2 TSW-133-07-H-S, U1 STM32WB15CCU6, X1 32 MHz, X2 32.768 kHz

Commit message: Temp
Other:
- sheet  RF & Power  renamed RF & Power
- moved on the sheet: R2
Changed lines of the file:
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@@
     (stroke (width 0) (type default))
   )
-  (wire (pts (xy 82.042 171.958) (xy 82.042 174.752))
+  (wire (pts (xy 82.042 171.958) (xy 82.042 176.022))
     (stroke (width 0) (type default))
   )
@@
     (stroke (width 0) (type default))
   )
-  (wire (pts (xy 82.042 182.372) (xy 82.042 187.452))
+  (wire (pts (xy 82.042 183.642) (xy 82.042 187.452))
     (stroke (width 0) (type default))
   )
@@
     )
   )
-  (symbol (lib_id "Device:R_US") (at 82.042 178.562 180) (unit 1)
-    (in_bom yes) (on_board yes) (dnp no)
-    (property "Reference" "R2" (at 79.756 178.562 90)
-      (effects (font (size 1.27 1.27)))
-    )
-    (property "Value" "10k" (at 84.582 178.816 90)
-      (effects (font (size 1.27 1.27)))
-    )
-    (property "Footprint" "Resistor_SMD:R_1218_3246Metric_Pad1.22x4.75mm_HandSolder" (at 89.916 181.864 90)
-      (effects (font (size 1.27 1.27)) hide)
-    )
-    (property "Datasheet" "~" (at 82.042 178.562 0)
+  (symbol (lib_id "Device:R_US") (at 82.042 179.832 180) (unit 1)
+    (in_bom yes) (on_board yes) (dnp no)
+    (property "Reference" "R2" (at 79.756 179.832 90)
+      (effects (font (size 1.27 1.27)))
+    )
+    (property "Value" "10k" (at 84.582 180.086 90)
+      (effects (font (size 1.27 1.27)))
+    )
+    (property "Footprint" "Resistor_SMD:R_1218_3246Metric_Pad1.22x4.75mm_HandSolder" (at 89.916 183.134 90)
+      (effects (font (size 1.27 1.27)) hide)
+    )
+    (property "Datasheet" "~" (at 82.042 179.832 0)
       (effects (font (size 1.27 1.27)) hide)
     )
@@
     (stroke (width 0.1524) (type solid))
     (fill (color 0 0 0 0.0000))
-    (property "Sheetname" " RF & Power " (at 257.302 125.476 0)
+    (property "Sheetname" "RF & Power" (at 257.81 125.476 0)
       (effects (font (size 1.27 1.27)) (justify left bottom))
     )

Commit message: Temp
Parts:
- C7: footprint Capacitor_SMD:C_01005_0402Metric -> Capacitor_THT:CP_Radial_D5.0mm_P2.00mm
Changed lines of the file:
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@@
       (effects (font (size 1.27 1.27)) (justify left))
     )
-    (property "Footprint" "Capacitor_SMD:C_01005_0402Metric" (at 21.5392 141.732 0)
+    (property "Footprint" "Capacitor_THT:CP_Radial_D5.0mm_P2.00mm" (at 21.5392 141.732 0)
       (effects (font (size 1.27 1.27)) hide)
     )

Commit message: Temp
Parts:
- added S1: USER BUTTON, TS026670BK160LCRD, symbol TS02-66-70-BK-160-LCR-D:TS02-66-70-BK-160-LCR-D
Connections:
- no-connect marks 3 -> 5
Changed lines of the file:
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@@
   )
   (no_connect (at 181.356 92.964))
+  (no_connect (at 220.98 131.826))
   (no_connect (at 181.356 90.424))
+  (no_connect (at 190.5 134.366))
   (no_connect (at 181.356 87.884))
   (wire (pts (xy 112.268 170.434) (xy 103.378 170.434))
@@
         )
       )
+    )
+  )
+  (symbol (lib_id "TS02-66-70-BK-160-LCR-D:TS02-66-70-BK-160-LCR-D") (at 190.5 131.826 0) (unit 1)
+    (in_bom yes) (on_board yes) (dnp no)
+    (property "Reference" "S1" (at 205.994 127.762 0)
+      (effects (font (size 1.27 1.27)))
+    )
+    (property "Value" "USER BUTTON" (at 205.994 138.43 0)
+      (effects (font (size 1.27 1.27)))
+    )
+    (property "Footprint" "TS026670BK160LCRD" (at 217.17 226.746 0)
+      (effects (font (size 1.27 1.27)) (justify left top) hide)
+    )
+    (property "Datasheet" "https://www.cuidevices.com/product/resource/ts02.pdf" (at 217.17 326.746 0)
+      (effects (font (size 1.27 1.27)) (justify left top) hide)
+    )
+    (property "Height" "7.2" (at 217.17 526.746 0)
+      (effects (font (size 1.27 1.27)) (justify left top) hide)
+    )
+    (property "Manufacturer_Name" "CUI Devices" (at 217.17 626.746 0)
+      (effects (font (size 1.27 1.27)) (justify left top) hide)
+    )
+    (property "Manufacturer_Part_Number" "TS02-66-70-BK-160-LCR-D" (at 217.17 726.746 0)
+      (effects (font (size 1.27 1.27)) (justify left top) hide)
+    )
+    (property "Mouser Part Number" "179-TS026670BK160LCR" (at 217.17 826.746 0)
+      (effects (font (size 1.27 1.27)) (justify left top) hide)
+    )
+    (property "Mouser Price/Stock" "https://www.mouser.co.uk/ProductDetail/CUI-Devices/TS02-66-70-BK-160-LCR-D?qs=A6eO%252BMLsxmSQ8aVkS4Cu7Q%3D%3D" (at 217.17 926.746 0)
+      (effects (font (size 1.27 1.27)) (justify left top) hide)
+    )
+    (property "Arrow Part Number" "TS02-66-70-BK-160-LCR-D" (at 217.17 1026.746 0)
+      (effects (font (size 1.27 1.27)) (justify left top) hide)
+    )
+    (property "Arrow Price/Stock" "https://www.arrow.com/en/products/ts02-66-70-bk-160-lcr-d/cui-devices?region=nac" (at 217.17 1126.746 0)
+      (effects (font (size 1.27 1.27)) (justify left top) hide)
+    )
+    (pin "3")
+    (pin "2")
+    (pin "1")
+    (pin "4")
+    (instances
+      (project "STM32WB breakout board"
+        (path "/29424def-bd0e-47af-8787-429d3d525da1"
+          (reference "S1") (unit 1)
+        )
+      )

Commit message: Temp
Parts:
- removed R3: 100k, Resistor_SMD:R_1218_3246Metric_Pad1.22x4.75mm_HandSolder, symbol Device:R_US
- added S2: RESET, TS026670BK160LCRD, symbol TS02-66-70-BK-160-LCR-D:TS02-66-70-BK-160-LCR-D
Connections:
- net GND: now also S1.4 (COM_2), S2.4 (COM_2)
- net NRST: now also S2.1 (NO_1)
- net PA1: no longer U1.10 (PA1)
- net USR_BTN: now reaches S1.1 (NO_1)
- net USR_BTN: now also U1.10 (PA1)
- no-connect marks 5 -> 7
Other:
- moved on the sheet: C18, D1, S1

Commit message: Switch updated
Parts:
- added C17: 100nF, Capacitor_SMD:C_0402_1005Metric, symbol Device:C
- added R1: 1k, Resistor_SMD:R_1218_3246Metric_Pad1.22x4.75mm_HandSolder, symbol Device:R_US
- added R3: 100k, Resistor_SMD:R_1218_3246Metric_Pad1.22x4.75mm_HandSolder, symbol Device:R_US
Connections:
- net 3V3: now also J1.21, J1.31, J1.32, R1.2; no longer J1.10, J1.18, J1.23
- net GND: now also J1.18, C17.2, R3.1; no longer S1.4 (COM_2)
- net NRST_Pin: now also J1.22; no longer J2.18
- net PA0: now also J2.01; no longer J2.16
- net PA1: now also J2.02; no longer J2.15
- net PA10: now also J1.33; no longer J1.22
- net PA11: now also J1.23; no longer J1.21
- net PA12: now also J2.15; no longer J1.20
- net PA15: now also J1.24; no longer J1.16
- net PB3: now also J1.25; no longer J1.15
- net PB4: now also J1.26; no longer J1.14
- net PB5: now also J1.27; no longer J1.13
- net PB6: now also J1.29; no longer J1.12
- net PB7: now also J1.30; no longer J1.11
- net PB8: now also J2.04; no longer J2.20
- net PB9: now also J2.03; no longer J2.19
- net SWCLK: now also J1.19; no longer J1.17
- net SWDIO: now also J1.20; no longer J1.19
- net USR_BTN: now also S1.4 (COM_2), C17.1, R3.2; no longer S1.1 (NO_1)
- net at S1.2 (NO_2): now also R1.1
- no-connect marks 7 -> 25
Other:
- moved on the sheet: S1, S2

Commit message: Pinout updated
Parts:
- removed J1, J2: TSW-133-07-H-S, SAMTEC_TSW-133-07-H-S, symbol TSW-133-07-H-S:TSW-133-07-H-S
- added J1, J2: Conn_02x10_Counter_Clockwise, Connector_PinSocket_2.54mm:PinSocket_2x10_P2.54mm_Vertical, symbol Connector_Generic:Conn_02x10_Counter_Clockwise
Connections:
- net PA4 is gone; now on net USR_BTN: U1.13 (PA4)
- net 3V3: now also J1.1 (Pin_1)
- net GND: now also J1.20 (Pin_20), J1.3 (Pin_3)
- net NRST_Pin: now also J1.2 (Pin_2)
- net PA0: now also J1.17 (Pin_17)
- net PA15: now also J1.8 (Pin_8)
- net PA7: now also J1.4 (Pin_4)
- net PA8: now also J1.5 (Pin_5)
- net PB2: now also J2.1 (Pin_1)
- net PB3: now also J2.2 (Pin_2)
- net PB4: now also J2.3 (Pin_3)
- net PB5: now also J2.4 (Pin_4)
- net PB6: now also J2.5 (Pin_5)
- net PB7: now also J2.6 (Pin_6)
- net PE4: now also J2.9 (Pin_9)
- net SWCLK: now also J1.18 (Pin_18)
- net SWDIO: now also J1.19 (Pin_19)
- net USR_BTN: no longer U1.10 (PA1)
- net PA10 renamed UART_RX/PA10
- net UART_RX/PA10: now also J1.7 (Pin_7)
- net PA11 renamed USB_N
- net USB_N: now also J1.10 (Pin_10)
- net PA12 renamed USB_P
- net USB_P: now also J1.9 (Pin_9)
- net PA2 renamed LPUART_TX/PA2
- net LPUART_TX/PA2: now also J1.15 (Pin_15)
- net PA3 renamed LPUART_RX/PA3
- net LPUART_RX/PA3: now also J1.14 (Pin_14)
- net PA5 renamed MOSI/PA5
- net MOSI/PA5: now also J1.12 (Pin_12)
- net PA6 renamed MISO/PA6
- net MISO/PA6: now also J1.11 (Pin_11)
- net PA9 renamed UART_TX/PA9
- net UART_TX/PA9: now also J1.6 (Pin_6)
- net PB8 renamed PB8/SCL
- net PB8/SCL: now also J2.7 (Pin_7)
- net PB9 renamed PB9/SDA
- net PB9/SDA: now also J2.8 (Pin_8)
- new net SCK/PA1: J1.16 (Pin_16), U1.10 (PA1)
- no-connect marks 25 -> 7

Commit message: Pinout updated
Changed lines of the file:
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@@
-    (stroke (width 0) (type default))
-  )
-  (wire (pts (xy 188.468 71.882) (xy 192.024 71.882))
     (stroke (width 0) (type default))
   )
@@
     (stroke (width 0) (type default))
   )
-  (wire (pts (xy 188.468 77.724) (xy 188.468 77.216))
-    (stroke (width 0) (type default))
-  )
   (wire (pts (xy 18.796 186.436) (xy 18.796 187.706))
     (stroke (width 0) (type default))
@@
     (stroke (width 0) (type default))
   )
-  (wire (pts (xy 188.468 74.422) (xy 192.024 74.422))
-    (stroke (width 0) (type default))
-  )
   (wire (pts (xy 89.662 171.958) (xy 82.042 171.958))
     (stroke (width 0) (type default))
@@
     (stroke (width 0) (type default))
   )
-  (wire (pts (xy 188.468 77.216) (xy 192.278 77.216))
-    (stroke (width 0) (type default))
-  )
   (wire (pts (xy 82.042 171.958) (xy 82.042 176.022))
     (stroke (width 0) (type default))
@@
     (stroke (width 0) (type default))
   )
-  (wire (pts (xy 188.468 72.644) (xy 188.468 71.882))
-    (stroke (width 0) (type default))
-  )
   (wire (pts (xy 82.042 183.642) (xy 82.042 187.452))
     (stroke (width 0) (type default))
@@
     (stroke (width 0) (type default))
   )
-  (wire (pts (xy 188.468 80.264) (xy 188.468 79.502))
-    (stroke (width 0) (type default))
-  )
   (wire (pts (xy 105.918 90.424) (xy 115.316 90.424))
     (stroke (width 0) (type default))
@@
     (stroke (width 0) (type default))
   )
-  (wire (pts (xy 181.356 72.644) (xy 188.468 72.644))
-    (stroke (width 0) (type default))
-  )
   (wire (pts (xy 181.356 34.544) (xy 183.769 34.544))
     (stroke (width 0) (type default))
@@
     (stroke (width 0) (type default))
   )
-  (wire (pts (xy 181.356 75.184) (xy 188.468 75.184))
-    (stroke (width 0) (type default))
-  )
   (wire (pts (xy 20.574 144.018) (xy 32.004 144.018))
     (stroke (width 0) (type default))
@@
     (stroke (width 0) (type default))
   )
-  (wire (pts (xy 181.356 80.264) (xy 188.468 80.264))
-    (stroke (width 0) (type default))
-  )
   (wire (pts (xy 105.156 77.724) (xy 115.316 77.724))
     (stroke (width 0) (type default))
@@
     (stroke (width 0) (type default))
   )
-  (wire (pts (xy 188.468 79.502) (xy 192.278 79.502))
-    (stroke (width 0) (type default))
-  )
-  (wire (pts (xy 188.468 75.184) (xy 188.468 74.422))
-    (stroke (width 0) (type default))
-  )
   (wire (pts (xy 23.622 173.228) (xy 18.796 173.228))
     (stroke (width 0) (type default))
@@
   )
   (wire (pts (xy 216.916 138.684) (xy 224.028 138.684))
-    (stroke (width 0) (type default))
-  )
-  (wire (pts (xy 181.356 77.724) (xy 188.468 77.724))
     (stroke (width 0) (type default))
   )
@@
     )
   )
-  (hierarchical_label "VFBSMPS" (shape input) (at 192.278 79.502 0) (fields_autoplaced)
-    (effects (font (size 1.27 1.27)) (justify left))
-  )
-  (hierarchical_label "VLXSMPS" (shape input) (at 192.024 74.422 0) (fields_autoplaced)
+  (hierarchical_label "VFBSMPS" (shape input) (at 181.356 80.264 0) (fields_autoplaced)
+    (effects (font (size 1.27 1.27)) (justify left))
+  )
+  (hierarchical_label "VLXSMPS" (shape input) (at 181.356 75.184 0) (fields_autoplaced)
     (effects (font (size 1.27 1.27)) (justify left))
   )
@@
     (effects (font (size 1.27 1.27)) (justify right))
   )
-  (hierarchical_label "VDDSMPS" (shape input) (at 192.024 71.882 0) (fields_autoplaced)
+  (hierarchical_label "VDDSMPS" (shape input) (at 181.356 72.644 0) (fields_autoplaced)
     (effects (font (size 1.27 1.27)) (justify left))
   )
@@
     (effects (font (size 1.27 1.27)) (justify right))
   )
-  (hierarchical_label "VSSSMPS" (shape input) (at 192.278 77.216 0) (fields_autoplaced)
-    (effects (font (size 1.27 1.27)) (justify left))
-  )
+  (hierarchical_label "VSSSMPS" (shape input) (at 181.356 77.724 0) (fields_autoplaced)
+    (effects (font (size 1.27 1.27)) (justify left))
+  )

Commit message: PCB layout updated
Parts:
- added J4, J5: Conn_02x10_Counter_Clockwise, Connector_PinSocket_2.54mm:PinSocket_2x10_P2.54mm_Vertical, symbol Connector_Generic:Conn_02x10_Counter_Clockwise
Connections:
- net 3V3: now also J4.1 (Pin_1)
- net GND: now also J4.20 (Pin_20), J4.3 (Pin_3)
- net LPUART_RX/PA3: now also J4.14 (Pin_14)
- net LPUART_TX/PA2: now also J4.15 (Pin_15)
- net MISO/PA6: now also J4.11 (Pin_11)
- net MOSI/PA5: now also J4.12 (Pin_12)
- net NRST_Pin: now also J4.2 (Pin_2)
- net PA0: now also J4.17 (Pin_17)
- net PA15: now also J4.8 (Pin_8)
- net PA7: now also J4.4 (Pin_4)
- net PA8: now also J4.5 (Pin_5)
- net PB2: now also J5.1 (Pin_1)
- net PB3: now also J5.2 (Pin_2)
- net PB4: now also J5.3 (Pin_3)
- net PB5: now also J5.4 (Pin_4)
- net PB6: now also J5.5 (Pin_5)
- net PB7: now also J5.6 (Pin_6)
- net PB8/SCL: now also J5.7 (Pin_7)
- net PB9/SDA: now also J5.8 (Pin_8)
- net PE4: now also J1.13 (Pin_13), J4.13 (Pin_13); no longer J2.9 (Pin_9)
- net SCK/PA1: now also J4.16 (Pin_16)
- net SWCLK: now also J4.18 (Pin_18)
- net SWDIO: now also J4.19 (Pin_19)
- net UART_RX/PA10: now also J4.7 (Pin_7)
- net UART_TX/PA9: now also J4.6 (Pin_6)
- net USB_N: now also J4.10 (Pin_10)
- net USB_P: now also J4.9 (Pin_9)
Other:
- moved on the sheet: C15, C16
