File: STM32WB breakout board/STM32WB breakout board.kicad_sch (KiCad schematic)
At the start: 25 parts, among them J1 Conn_02x10_Counter_Clockwise, J2 Conn_02x10_Counter_Clockwise, J4 Conn_02x10_Counter_Clockwise, J5 Conn_02x10_Counter_Clockwise, U1 STM32WB15CCU6, X1 32 MHz, X2 32.768 kHz

Commit message: PCB updated
Changed lines of the file:
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@@
   (junction (at 45.212 132.08) (diameter 0) (color 0 0 0 0)
   )
-  (junction (at 101.854 132.969) (diameter 0) (color 0 0 0 0)
-  )
   (junction (at 35.052 173.228) (diameter 0) (color 0 0 0 0)
   )
@@
   (junction (at 107.95 144.272) (diameter 0) (color 0 0 0 0)
   )
+  (junction (at 113.538 132.588) (diameter 0) (color 0 0 0 0)
+  )
   (junction (at 207.01 120.142) (diameter 0) (color 0 0 0 0)
   )
@@
   (junction (at 32.004 132.08) (diameter 0) (color 0 0 0 0)
   )
+  (junction (at 101.854 132.588) (diameter 0) (color 0 0 0 0)
+  )
   (junction (at 213.868 132.08) (diameter 0) (color 0 0 0 0)
   )
@@
   )
   (junction (at 20.574 132.08) (diameter 0) (color 0 0 0 0)
-  )
-  (junction (at 113.538 132.969) (diameter 0) (color 0 0 0 0)
   )
   (junction (at 32.004 144.018) (diameter 0) (color 0 0 0 0)
@@
     (stroke (width 0) (type default))
   )
+  (wire (pts (xy 113.538 132.588) (xy 116.586 132.588))
+    (stroke (width 0) (type default))
+  )
   (wire (pts (xy 43.18 45.72) (xy 46.228 45.72))
     (stroke (width 0) (type default))
@@
     (stroke (width 0) (type default))
   )
-  (wire (pts (xy 113.538 132.969) (xy 119.634 132.969))
-    (stroke (width 0) (type default))
-  )
   (wire (pts (xy 18.796 173.228) (xy 18.796 178.816))
     (stroke (width 0) (type default))
@@
     (stroke (width 0) (type default))
   )
+  (wire (pts (xy 101.854 132.588) (xy 101.854 134.747))
+    (stroke (width 0) (type default))
+  )
   (wire (pts (xy 60.198 168.148) (xy 60.198 172.466))
     (stroke (width 0) (type default))
@@
     (stroke (width 0) (type default))
   )
-  (wire (pts (xy 101.854 132.969) (xy 101.854 134.747))
-    (stroke (width 0) (type default))
-  )
   (wire (pts (xy 35.052 167.386) (xy 35.052 173.228))
     (stroke (width 0) (type default))
@@
     (stroke (width 0) (type default))
   )
-  (wire (pts (xy 101.854 132.969) (xy 113.538 132.969))
+  (wire (pts (xy 101.854 132.588) (xy 113.538 132.588))
     (stroke (width 0) (type default))
   )
@@
     (stroke (width 0) (type default))
   )
-  (wire (pts (xy 101.854 128.778) (xy 101.854 132.969))
+  (wire (pts (xy 101.854 128.778) (xy 101.854 132.588))
     (stroke (width 0) (type default))
   )
@@
     (stroke (width 0) (type default))
   )
-  (wire (pts (xy 113.538 134.62) (xy 113.538 132.969))
+  (wire (pts (xy 113.538 134.62) (xy 113.538 132.588))
     (stroke (width 0) (type default))
   )
@@
     (effects (font (size 1.27 1.27)) (justify left bottom))
   )
-  (label "VDDA" (at 119.634 132.969 0) (fields_autoplaced)
-    (effects (font (size 1.27 1.27)) (justify left bottom))
-  )
+  (label "VDDA" (at 116.586 132.588 0) (fields_autoplaced)
+    (effects (font (size 1.27 1.27)) (justify left bottom))
+  )

Commit message: PCB updated
Other:
- moved on the sheet: R3
Changed lines of the file:
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@@
     (date "2023-12-16")
   )
+  (junction (at 207.01 120.142) (diameter 0) (color 0 0 0 0)
+  )
   (junction (at 66.802 132.08) (diameter 0) (color 0 0 0 0)
   )
@@
   )
   (junction (at 113.538 132.588) (diameter 0) (color 0 0 0 0)
-  )
-  (junction (at 207.01 120.142) (diameter 0) (color 0 0 0 0)
   )
   (junction (at 56.642 132.08) (diameter 0) (color 0 0 0 0)
@@
     (stroke (width 0) (type default))
   )
-  (wire (pts (xy 207.01 120.142) (xy 220.98 120.142))
-    (stroke (width 0) (type default))
-  )
   (wire (pts (xy 224.536 36.068) (xy 227.076 36.068))
     (stroke (width 0) (type default))
@@
     (stroke (width 0) (type default))
   )
-  (wire (pts (xy 220.98 132.08) (xy 220.98 129.794))
+  (wire (pts (xy 219.456 132.08) (xy 219.456 129.794))
     (stroke (width 0) (type default))
   )
@@
     (stroke (width 0) (type default))
   )
-  (wire (pts (xy 220.98 120.142) (xy 220.98 122.174))
+  (wire (pts (xy 219.456 120.142) (xy 219.456 122.174))
     (stroke (width 0) (type default))
   )
@@
     (stroke (width 0) (type default))
   )
+  (wire (pts (xy 202.692 120.142) (xy 207.01 120.142))
+    (stroke (width 0) (type default))
+  )
   (wire (pts (xy 35.052 167.386) (xy 35.052 173.228))
     (stroke (width 0) (type default))
@@
     (stroke (width 0) (type default))
   )
-  (wire (pts (xy 202.692 120.142) (xy 207.01 120.142))
-    (stroke (width 0) (type default))
-  )
   (wire (pts (xy 37.338 38.1) (xy 46.228 38.1))
     (stroke (width 0) (type default))
@@
     (stroke (width 0) (type default))
   )
+  (wire (pts (xy 207.01 120.142) (xy 219.456 120.142))
+    (stroke (width 0) (type default))
+  )
   (wire (pts (xy 45.212 144.018) (xy 45.212 149.098))
     (stroke (width 0) (type default))
@@
     (stroke (width 0) (type default))
   )
-  (wire (pts (xy 213.868 132.08) (xy 220.98 132.08))
+  (wire (pts (xy 213.868 132.08) (xy 219.456 132.08))
     (stroke (width 0) (type default))
   )
@@
     (effects (font (size 1.27 1.27)) (justify left bottom))
   )
-  (label "USR_BTN" (at 214.376 120.142 180) (fields_autoplaced)
-    (effects (font (size 1.27 1.27)) (justify right bottom))
+  (label "USR_BTN" (at 204.978 120.142 0) (fields_autoplaced)
+    (effects (font (size 1.27 1.27)) (justify left bottom))
   )
   (label "NRST_Pin" (at 43.18 35.56 180) (fields_autoplaced)
@@
     )
   )
-  (symbol (lib_id "Device:R_US") (at 220.98 125.984 180) (unit 1)
+  (symbol (lib_id "Device:R_US") (at 219.456 125.984 180) (unit 1)
     (in_bom yes) (on_board yes) (dnp no)
-    (property "Reference" "R3" (at 218.694 125.984 90)
+    (property "Reference" "R3" (at 217.17 125.984 90)
       (effects (font (size 1.27 1.27)))
     )
-    (property "Value" "100k" (at 223.52 126.238 90)
+    (property "Value" "100k" (at 221.996 126.238 90)
       (effects (font (size 1.27 1.27)))
     )
-    (property "Footprint" "Resistor_SMD:R_1206_3216Metric" (at 228.854 129.286 90)
-      (effects (font (size 1.27 1.27)) hide)
-    )
-    (property "Datasheet" "~" (at 220.98 125.984 0)
-      (effects (font (size 1.27 1.27)) hide)
-    )
+    (property "Footprint" "Resistor_SMD:R_1206_3216Metric" (at 227.33 129.286 90)
+      (effects (font (size 1.27 1.27)) hide)
+    )
+    (property "Datasheet" "~" (at 219.456 125.984 0)
+      (effects (font (size 1.27 1.27)) hide)
+    )
