File: STM32WB breakout board/ RF Section_sch.kicad_sch (KiCad schematic)
At the start: 7 parts, among them J3 RSP-122811-02

Commit message: Temp
Parts:
- added C4: 4.7 uF, Capacitor_THT:C_Radial_D5.0mm_H11.0mm_P2.00mm, symbol Device:C
- added C4: 100nF, Capacitor_THT:C_Radial_D5.0mm_H11.0mm_P2.00mm, symbol Device:C
Connections:
- net 3V3: now also C4.1, C4.1
- net GND: now also C4.2, C4.2
Other:
- moved on the sheet: C3, C4, C7, C9, FL1, J3, L1

Commit message: Temp
Parts:
- added C4: 4.7 uF, Capacitor_THT:C_Radial_D5.0mm_H11.0mm_P2.00mm, symbol Device:C
- added L2: LQM21FN100M70L, LQM21FN100M70L:INDC2012X145N, symbol LQM21FN100M70L:LQM21FN100M70L
- added L3: LQG15WZ10NJ02D, LQG15WZ10NJ02D:INDC1006X60N, symbol LQG15WZ10NJ02D:LQG15WZ10NJ02D
Connections:
- net GND: now also C4.2
- net VLXSMPS: now also L3.2
- new net: L2.2, L3.1
- new net VFBSMPS: C4.1, L2.1
Other:
- note added: "10 nH"
- note added: "10 uH"
- moved on the sheet: C3, C4

Commit message: Temp
Parts:
- removed C4: 100nF, Capacitor_THT:C_Radial_D5.0mm_H11.0mm_P2.00mm, symbol Device:C
- added C11: 100nF, Capacitor_SMD:C_0402_1005Metric, symbol Device:C
- C3: footprint Capacitor_THT:C_Radial_D5.0mm_H11.0mm_P2.00mm -> Capacitor_SMD:C_0402_1005Metric
- renumbered C9 to C3, C7 to C4
Connections:
- net 3V3: now also C11.1
- net GND: now also C11.2
Changed lines of the file:
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@@
   (symbol (lib_id "GRM1555C1HR80BA01D:GRM1555C1HR80BA01D") (at 64.516 54.864 90) (unit 1)
     (in_bom yes) (on_board yes) (dnp no)
-    (property "Reference" "C9" (at 57.404 52.07 90)
+    (property "Reference" "C3" (at 57.404 52.07 90)
       (effects (font (size 1.27 1.27)) (justify right))
     )
@@
       (project "STM32WB breakout board"
         (path "/29424def-bd0e-47af-8787-429d3d525da1/1e4823cc-51de-4557-be75-82cccb133913"
-          (reference "C9") (unit 1)
+          (reference "C3") (unit 1)
         )
       )
@@
   (symbol (lib_id "GRM1555C1HR30WA01D:GRM1555C1HR30WA01D") (at 85.598 53.848 90) (unit 1)
     (in_bom yes) (on_board yes) (dnp no) (fields_autoplaced)
-    (property "Reference" "C7" (at 89.408 51.308 90)
+    (property "Reference" "C4" (at 88.9 51.308 90)
       (effects (font (size 1.27 1.27)) (justify right))
     )
-    (property "Value" "GRM1555C1HR30WA01D" (at 89.408 53.848 90)
+    (property "Value" "GRM1555C1HR30WA01D" (at 88.9 53.848 90)
       (effects (font (size 1.27 1.27)) (justify right))
     )
@@
       (project "STM32WB breakout board"
         (path "/29424def-bd0e-47af-8787-429d3d525da1/1e4823cc-51de-4557-be75-82cccb133913"
-          (reference "C7") (unit 1)
+          (reference "C4") (unit 1)
+        )
+      )
+    )
+  )
+  (symbol (lib_id "Device:C") (at 117.856 106.934 0) (unit 1)
+    (in_bom yes) (on_board yes) (dnp no)
+    (property "Reference" "C11" (at 119.634 104.648 0)
+      (effects (font (size 1.27 1.27)) (justify left))
+    )
+    (property "Value" "100nF" (at 118.872 110.49 0)
+      (effects (font (size 1.27 1.27)) (justify left))
+    )
+    (property "Footprint" "Capacitor_SMD:C_0402_1005Metric" (at 118.8212 110.744 0)
+      (effects (font (size 1.27 1.27)) hide)
+    )
+    (property "Datasheet" "~" (at 117.856 106.934 0)
+      (effects (font (size 1.27 1.27)) hide)
+    )
+    (pin "2")
+    (pin "1")
+    (instances
+      (project "STM32WB breakout board"
+        (path "/29424def-bd0e-47af-8787-429d3d525da1"
+          (reference "C11") (unit 1)
+        )
+        (path "/29424def-bd0e-47af-8787-429d3d525da1/1e4823cc-51de-4557-be75-82cccb133913"
+          (reference "C13") (unit 1)
         )
       )
@@
       (effects (font (size 1.27 1.27)) (justify left))
     )
-    (property "Footprint" "Capacitor_THT:C_Radial_D5.0mm_H11.0mm_P2.00mm" (at 261.5692 33.02 0)
+    (property "Footprint" "Capacitor_SMD:C_0402_1005Metric" (at 261.5692 33.02 0)
       (effects (font (size 1.27 1.27)) hide)
     )
@@
         )
         (path "/29424def-bd0e-47af-8787-429d3d525da1/1e4823cc-51de-4557-be75-82cccb133913"
-          (reference "C6") (unit 1)
+          (reference "C2") (unit 1)
         )
       )
@@
         )
         (path "/29424def-bd0e-47af-8787-429d3d525da1/1e4823cc-51de-4557-be75-82cccb133913"
-          (reference "C10") (unit 1)
+          (reference "C17") (unit 1)
         )
       )
@@
         )
         (path "/29424def-bd0e-47af-8787-429d3d525da1/1e4823cc-51de-4557-be75-82cccb133913"
-          (reference "C1") (unit 1)
+          (reference "C12") (unit 1)
         )
       )
@@
     )
   )
-  (symbol (lib_id "Device:C") (at 117.856 106.934 0) (unit 1)
-    (in_bom yes) (on_board yes) (dnp no)
-    (property "Reference" "C4" (at 118.618 104.394 0)
-      (effects (font (size 1.27 1.27)) (justify left))
-    )
-    (property "Value" "100nF" (at 118.618 109.728 0)
-      (effects (font (size 1.27 1.27)) (justify left))
-    )
-    (property "Footprint" "Capacitor_THT:C_Radial_D5.0mm_H11.0mm_P2.00mm" (at 118.8212 110.744 0)
-      (effects (font (size 1.27 1.27)) hide)
-    )
-    (property "Datasheet" "~" (at 117.856 106.934 0)
+  (symbol (lib_id "power:GND") (at 135.128 20.066 180) (unit 1)
+    (in_bom yes) (on_board yes) (dnp no)
+    (property "Reference" "#PWR01" (at 135.128 13.716 0)
+      (effects (font (size 1.27 1.27)) hide)
+    )
+    (property "Value" "GND" (at 137.16 16.51 0)
+      (effects (font (size 1.27 1.27)) (justify left))
+    )
+    (property "Footprint" "" (at 135.128 20.066 0)
+      (effects (font (size 1.27 1.27)) hide)
+    )
+    (property "Datasheet" "" (at 135.128 20.066 0)
+      (effects (font (size 1.27 1.27)) hide)
+    )
+    (pin "1")
+    (instances
+      (project "STM32WB breakout board"
+        (path "/29424def-bd0e-47af-8787-429d3d525da1"
+          (reference "#PWR01") (unit 1)
+        )
+        (path "/29424def-bd0e-47af-8787-429d3d525da1/1e4823cc-51de-4557-be75-82cccb133913"
+          (reference "#PWR08") (unit 1)
+        )
+      )
+    )
+  )
+  (symbol (lib_id "power:GND") (at 117.856 115.062 0) (unit 1)
+    (in_bom yes) (on_board yes) (dnp no)
+    (property "Reference" "#PWR01" (at 117.856 121.412 0)
+      (effects (font (size 1.27 1.27)) hide)
+    )
+    (property "Value" "GND" (at 115.824 118.618 0)
+      (effects (font (size 1.27 1.27)) (justify left))
+    )
+    (property "Footprint" "" (at 117.856 115.062 0)
+      (effects (font (size 1.27 1.27)) hide)
+    )
+    (property "Datasheet" "" (at 117.856 115.062 0)
+      (effects (font (size 1.27 1.27)) hide)
+    )
+    (pin "1")
+    (instances
+      (project "STM32WB breakout board"
+        (path "/29424def-bd0e-47af-8787-429d3d525da1"
+          (reference "#PWR01") (unit 1)
+        )
+        (path "/29424def-bd0e-47af-8787-429d3d525da1/1e4823cc-51de-4557-be75-82cccb133913"
+          (reference "#PWR016") (unit 1)
+        )
+      )
+    )
+  )
+  (symbol (lib_id "Device:C") (at 246.888 29.21 0) (unit 1)
+    (in_bom yes) (on_board yes) (dnp no)
+    (property "Reference" "C4" (at 248.666 26.924 0)
+      (effects (font (size 1.27 1.27)) (justify left))
+    )
+    (property "Value" "100nF" (at 248.666 31.496 0)
+      (effects (font (size 1.27 1.27)) (justify left))
+    )
+    (property "Footprint" "Capacitor_THT:C_Radial_D5.0mm_H11.0mm_P2.00mm" (at 247.8532 33.02 0)
+      (effects (font (size 1.27 1.27)) hide)
+    )
+    (property "Datasheet" "~" (at 246.888 29.21 0)
       (effects (font (size 1.27 1.27)) hide)
     )
@@
         )
         (path "/29424def-bd0e-47af-8787-429d3d525da1/1e4823cc-51de-4557-be75-82cccb133913"
-          (reference "C8") (unit 1)
-        )
-      )
-    )
-  )
-  (symbol (lib_id "power:GND") (at 135.128 20.066 180) (unit 1)
-    (in_bom yes) (on_board yes) (dnp no)
-    (property "Reference" "#PWR01" (at 135.128 13.716 0)
-      (effects (font (size 1.27 1.27)) hide)
-    )
-    (property "Value" "GND" (at 137.16 16.51 0)
-      (effects (font (size 1.27 1.27)) (justify left))
-    )
-    (property "Footprint" "" (at 135.128 20.066 0)
-      (effects (font (size 1.27 1.27)) hide)
-    )
-    (property "Datasheet" "" (at 135.128 20.066 0)
-      (effects (font (size 1.27 1.27)) hide)
-    )
-    (pin "1")
-    (instances
-      (project "STM32WB breakout board"
-        (path "/29424def-bd0e-47af-8787-429d3d525da1"
-          (reference "#PWR01") (unit 1)
-        )
-        (path "/29424def-bd0e-47af-8787-429d3d525da1/1e4823cc-51de-4557-be75-82cccb133913"
-          (reference "#PWR08") (unit 1)
-        )
-      )
-    )
-  )
-  (symbol (lib_id "power:GND") (at 117.856 115.062 0) (unit 1)
-    (in_bom yes) (on_board yes) (dnp no)
-    (property "Reference" "#PWR01" (at 117.856 121.412 0)
-      (effects (font (size 1.27 1.27)) hide)
-    )
-    (property "Value" "GND" (at 115.824 118.618 0)
-      (effects (font (size 1.27 1.27)) (justify left))
-    )
-    (property "Footprint" "" (at 117.856 115.062 0)
-      (effects (font (size 1.27 1.27)) hide)
-    )
-    (property "Datasheet" "" (at 117.856 115.062 0)
-      (effects (font (size 1.27 1.27)) hide)
-    )
-    (pin "1")
-    (instances
-      (project "STM32WB breakout board"
-        (path "/29424def-bd0e-47af-8787-429d3d525da1"
-          (reference "#PWR01") (unit 1)
-        )
-        (path "/29424def-bd0e-47af-8787-429d3d525da1/1e4823cc-51de-4557-be75-82cccb133913"
-          (reference "#PWR016") (unit 1)
-        )
-      )
-    )
-  )
-  (symbol (lib_id "Device:C") (at 246.888 29.21 0) (unit 1)
-    (in_bom yes) (on_board yes) (dnp no)
-    (property "Reference" "C4" (at 248.666 26.924 0)
-      (effects (font (size 1.27 1.27)) (justify left))
-    )
-    (property "Value" "100nF" (at 248.666 31.496 0)
-      (effects (font (size 1.27 1.27)) (justify left))
-    )
-    (property "Footprint" "Capacitor_THT:C_Radial_D5.0mm_H11.0mm_P2.00mm" (at 247.8532 33.02 0)
-      (effects (font (size 1.27 1.27)) hide)
-    )
-    (property "Datasheet" "~" (at 246.888 29.21 0)
-      (effects (font (size 1.27 1.27)) hide)
-    )
-    (pin "2")
-    (pin "1")
-    (instances
-      (project "STM32WB breakout board"
-        (path "/29424def-bd0e-47af-8787-429d3d525da1"
-          (reference "C4") (unit 1)
-        )
-        (path "/29424def-bd0e-47af-8787-429d3d525da1/1e4823cc-51de-4557-be75-82cccb133913"
-          (reference "C5") (unit 1)
-        )
-      )
+          (reference "C1") (unit 1)
+        )
+      )

Commit message: Temp
Parts:
- renumbered L3 to L2, L2 to L3
Other:
- note added: "2.7 nH"
- note removed: "RF Inductor"
Changed lines of the file:
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@@
     (effects (font (size 1.27 1.27)) (justify left bottom))
   )
-  (text "RF Inductor\n" (at 69.596 44.196 0)
+  (text "2.7 nH\n" (at 71.374 44.196 0)
     (effects (font (size 1.27 1.27)) (justify left bottom))
   )
@@
   )
   (symbol (lib_id "LQM21FN100M70L:LQM21FN100M70L") (at 28.448 105.156 90) (unit 1)
-    (in_bom yes) (on_board yes) (dnp no) (fields_autoplaced)
-    (property "Reference" "L2" (at 22.352 105.156 0)
-      (effects (font (size 1.27 1.27)))
-    )
-    (property "Value" "LQM21FN100M70L" (at 24.892 105.156 0)
-      (effects (font (size 1.27 1.27)))
+    (in_bom yes) (on_board yes) (dnp no)
+    (property "Reference" "L3" (at 23.368 103.886 0)
+      (effects (font (size 1.27 1.27)) (justify right))
+    )
+    (property "Value" "LQM21FN100M70L" (at 25.654 96.774 0)
+      (effects (font (size 1.27 1.27)) (justify right))
     )
     (property "Footprint" "LQM21FN100M70L:INDC2012X145N" (at 28.448 105.156 0)
@@
       (project "STM32WB breakout board"
         (path "/29424def-bd0e-47af-8787-429d3d525da1/1e4823cc-51de-4557-be75-82cccb133913"
-          (reference "L2") (unit 1)
+          (reference "L3") (unit 1)
         )
       )
@@
   (symbol (lib_id "LQG15WZ10NJ02D:LQG15WZ10NJ02D") (at 44.196 93.726 0) (unit 1)
     (in_bom yes) (on_board yes) (dnp no) (fields_autoplaced)
-    (property "Reference" "L3" (at 44.196 87.63 0)
+    (property "Reference" "L2" (at 44.196 87.63 0)
       (effects (font (size 1.27 1.27)))
     )
@@
       (project "STM32WB breakout board"
         (path "/29424def-bd0e-47af-8787-429d3d525da1/1e4823cc-51de-4557-be75-82cccb133913"
-          (reference "L3") (unit 1)
-        )
-      )
+          (reference "L2") (unit 1)
+        )
+      )

Commit message: Temp
Parts:
- C4: footprint Capacitor_THT:C_Radial_D5.0mm_H11.0mm_P2.00mm -> Capacitor_SMD:C_0402_1005Metric
Changed lines of the file:
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@@
       (effects (font (size 1.27 1.27)) (justify left))
     )
-    (property "Footprint" "Capacitor_THT:C_Radial_D5.0mm_H11.0mm_P2.00mm" (at 247.8532 33.02 0)
+    (property "Footprint" "Capacitor_SMD:C_0402_1005Metric" (at 247.8532 33.02 0)
       (effects (font (size 1.27 1.27)) hide)
     )

Commit message: Temp
Parts:
- C4: footprint Capacitor_THT:C_Radial_D5.0mm_H11.0mm_P2.00mm -> Capacitor_SMD:C_01005_0402Metric
Changed lines of the file:
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@@
       (effects (font (size 1.27 1.27)) (justify left))
     )
-    (property "Footprint" "Capacitor_THT:C_Radial_D5.0mm_H11.0mm_P2.00mm" (at 29.4132 125.476 0)
+    (property "Footprint" "Capacitor_SMD:C_01005_0402Metric" (at 29.4132 125.476 0)
       (effects (font (size 1.27 1.27)) hide)
     )
@@
         (path "/29424def-bd0e-47af-8787-429d3d525da1/1e4823cc-51de-4557-be75-82cccb133913"
           (reference "L3") (unit 1)
-        )
-      )
-    )
-  )
-  (symbol (lib_id "Device:C") (at 103.378 107.188 0) (unit 1)
-    (in_bom yes) (on_board yes) (dnp no)
-    (property "Reference" "C4" (at 104.394 105.156 0)
-      (effects (font (size 1.27 1.27)) (justify left))
-    )
-    (property "Value" "4.7 uF" (at 104.14 109.982 0)
-      (effects (font (size 1.27 1.27)) (justify left))
-    )
-    (property "Footprint" "Capacitor_THT:C_Radial_D5.0mm_H11.0mm_P2.00mm" (at 104.3432 110.998 0)
-      (effects (font (size 1.27 1.27)) hide)
-    )
-    (property "Datasheet" "~" (at 103.378 107.188 0)
-      (effects (font (size 1.27 1.27)) hide)
-    )
-    (pin "2")
-    (pin "1")
-    (instances
-      (project "STM32WB breakout board"
-        (path "/29424def-bd0e-47af-8787-429d3d525da1"
-          (reference "C4") (unit 1)
-        )
-        (path "/29424def-bd0e-47af-8787-429d3d525da1/1e4823cc-51de-4557-be75-82cccb133913"
-          (reference "C12") (unit 1)
         )
       )
@@
         )
       )
+    )
+  )
+  (symbol (lib_id "Device:C") (at 103.378 107.188 0) (unit 1)
+    (in_bom yes) (on_board yes) (dnp no)
+    (property "Reference" "C4" (at 104.394 105.156 0)
+      (effects (font (size 1.27 1.27)) (justify left))
+    )
+    (property "Value" "4.7 uF" (at 104.14 109.982 0)
+      (effects (font (size 1.27 1.27)) (justify left))
+    )
+    (property "Footprint" "Capacitor_SMD:C_01005_0402Metric" (at 104.3432 110.998 0)
+      (effects (font (size 1.27 1.27)) hide)
+    )
+    (property "Datasheet" "~" (at 103.378 107.188 0)
+      (effects (font (size 1.27 1.27)) hide)
+    )
+    (pin "2")
+    (pin "1")
+    (instances
+      (project "STM32WB breakout board"
+        (path "/29424def-bd0e-47af-8787-429d3d525da1"
+          (reference "C4") (unit 1)
+        )
+        (path "/29424def-bd0e-47af-8787-429d3d525da1/1e4823cc-51de-4557-be75-82cccb133913"
+          (reference "C12") (unit 1)
+        )
+      )

Commit message: Temp
Other:
- note added: "*Replace with right angle SMA connector"
Changed lines of the file:
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@@
     (effects (font (size 2.54 2.54)) (justify left bottom))
+  )
+  (text "*Replace with right angle SMA connector" (at 184.658 48.768 0)
+    (effects (font (size 1.27 1.27)) (justify left bottom))
   )
   (text "10 nH\n" (at 41.656 96.774 0)

Commit message: Temp
Parts:
- removed C4 (x2): 4.7 uF, Capacitor_SMD:C_01005_0402Metric, symbol Device:C
- added C7 (x2): 4.7 uF, Capacitor_THT:CP_Radial_D5.0mm_P2.00mm, symbol Device:C
Connections:
- net 3V3: now also C7.1
- net GND: now also C7.2, C7.2
- net VFBSMPS: now also C7.1
Changed lines of the file:
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@@
+    )
+  )
+  (symbol (lib_id "Device:C") (at 103.378 107.188 0) (unit 1)
+    (in_bom yes) (on_board yes) (dnp no)
+    (property "Reference" "C7" (at 104.394 105.156 0)
+      (effects (font (size 1.27 1.27)) (justify left))
+    )
+    (property "Value" "4.7 uF" (at 104.14 109.982 0)
+      (effects (font (size 1.27 1.27)) (justify left))
+    )
+    (property "Footprint" "Capacitor_THT:CP_Radial_D5.0mm_P2.00mm" (at 104.3432 110.998 0)
+      (effects (font (size 1.27 1.27)) hide)
+    )
+    (property "Datasheet" "~" (at 103.378 107.188 0)
+      (effects (font (size 1.27 1.27)) hide)
+    )
+    (pin "2")
+    (pin "1")
+    (instances
+      (project "STM32WB breakout board"
+        (path "/29424def-bd0e-47af-8787-429d3d525da1"
+          (reference "C7") (unit 1)
+        )
+        (path "/29424def-bd0e-47af-8787-429d3d525da1/1e4823cc-51de-4557-be75-82cccb133913"
+          (reference "C12") (unit 1)
+        )
+      )
     )
   )
   (symbol (lib_id "Device:C") (at 28.448 121.666 0) (unit 1)
     (in_bom yes) (on_board yes) (dnp no)
-    (property "Reference" "C4" (at 29.464 119.634 0)
+    (property "Reference" "C7" (at 29.464 119.634 0)
       (effects (font (size 1.27 1.27)) (justify left))
     )
@@
       (effects (font (size 1.27 1.27)) (justify left))
     )
-    (property "Footprint" "Capacitor_SMD:C_01005_0402Metric" (at 29.4132 125.476 0)
+    (property "Footprint" "Capacitor_THT:CP_Radial_D5.0mm_P2.00mm" (at 29.4132 125.476 0)
       (effects (font (size 1.27 1.27)) hide)
     )
@@
       (project "STM32WB breakout board"
         (path "/29424def-bd0e-47af-8787-429d3d525da1"
-          (reference "C4") (unit 1)
-        )
-        (path "/29424def-bd0e-47af-8787-429d3d525da1/1e4823cc-51de-4557-be75-82cccb133913"
-          (reference "C17") (unit 1)
+          (reference "C7") (unit 1)
+        )
+        (path "/29424def-bd0e-47af-8787-429d3d525da1/1e4823cc-51de-4557-be75-82cccb133913"
+          (reference "C14") (unit 1)
         )
       )
@@
         )
       )
-    )
-  )
-  (symbol (lib_id "Device:C") (at 103.378 107.188 0) (unit 1)
-    (in_bom yes) (on_board yes) (dnp no)
-    (property "Reference" "C4" (at 104.394 105.156 0)
-      (effects (font (size 1.27 1.27)) (justify left))
-    )
-    (property "Value" "4.7 uF" (at 104.14 109.982 0)
-      (effects (font (size 1.27 1.27)) (justify left))
-    )
-    (property "Footprint" "Capacitor_SMD:C_01005_0402Metric" (at 104.3432 110.998 0)
-      (effects (font (size 1.27 1.27)) hide)
-    )
-    (property "Datasheet" "~" (at 103.378 107.188 0)
-      (effects (font (size 1.27 1.27)) hide)
-    )
-    (pin "2")
-    (pin "1")
-    (instances
-      (project "STM32WB breakout board"
-        (path "/29424def-bd0e-47af-8787-429d3d525da1"
-          (reference "C4") (unit 1)
-        )
-        (path "/29424def-bd0e-47af-8787-429d3d525da1/1e4823cc-51de-4557-be75-82cccb133913"
-          (reference "C12") (unit 1)
-        )
-      )
