File: STM32WB breakout board/_autosave-STM32WB breakout board.kicad_pcb (KiCad board)
At the start: 2 copper layers, 70 x 70 mm, 35 parts, among them J1 Conn_02x10_Counter_Clockwise, J2 Conn_02x10_Counter_Clockwise, J3 RSP-122811-02, U1 STM32WB15CCU6, X1 32 MHz, X2 32.768 kHz

Commit message: Pinout updated
Connections:
- J1 pad 10: unconnected-(J1-Pin_10-Pad10) -> /USB_N
- J1 pad 11: unconnected-(J1-Pin_11-Pad11) -> /PA6
- J1 pad 12: unconnected-(J1-Pin_12-Pad12) -> /PA5
- J1 pad 13: unconnected-(J1-Pin_13-Pad13) -> /PA4
- J1 pad 14: unconnected-(J1-Pin_14-Pad14) -> /PA3
- J1 pad 15: unconnected-(J1-Pin_15-Pad15) -> /PA2
- J1 pad 16: unconnected-(J1-Pin_16-Pad16) -> /PA1
- J1 pad 17: unconnected-(J1-Pin_17-Pad17) -> /PA0
- J1 pad 2: GND -> /NRST_Pin
- J1 pad 20: /NRST_Pin -> GND
- J1 pad 3: unconnected-(J1-Pin_3-Pad3) -> GND
- J1 pad 4: unconnected-(J1-Pin_4-Pad4) -> /PA7
- J1 pad 5: unconnected-(J1-Pin_5-Pad5) -> /PA8
- J1 pad 6: unconnected-(J1-Pin_6-Pad6) -> /PA9
- J1 pad 7: unconnected-(J1-Pin_7-Pad7) -> /PA10
- J1 pad 8: unconnected-(J1-Pin_8-Pad8) -> /PA15
- J1 pad 9: unconnected-(J1-Pin_9-Pad9) -> /USB_P
- J2 pad 1: unconnected-(J2-Pin_1-Pad1) -> /PB2
- J2 pad 2: unconnected-(J2-Pin_2-Pad2) -> /PB3
- J2 pad 3: unconnected-(J2-Pin_3-Pad3) -> /PB4
- J2 pad 4: unconnected-(J2-Pin_4-Pad4) -> /PB5
- J2 pad 5: unconnected-(J2-Pin_5-Pad5) -> /PB6
- J2 pad 6: unconnected-(J2-Pin_6-Pad6) -> /PB7
- J2 pad 7: unconnected-(J2-Pin_7-Pad7) -> /PB8
- J2 pad 8: unconnected-(J2-Pin_8-Pad8) -> /PB9
- J2 pad 9: unconnected-(J2-Pin_9-Pad9) -> /PE4
- U1 pad 37: /PA11 -> /USB_N
- U1 pad 38: /PA12 -> /USB_P
Routing:
- net /USB_P: track 0.00 -> 48.8 mm
- net /PA12: track 48.8 -> 0.00 mm
- net /USB_N: track 0.00 -> 39.3 mm
- net /PA11: track 39.3 -> 0.00 mm
